File: Power Supply LM2576/Power Supply LM2576.kicad_pcb (KiCad board)
At the start: 2 copper layers, 32 parts, among them J1 Power IN, J2 Conn_02x03_Odd_Even, J3 Power OUT, Q1 IRLML0030, U1 INA169, U2 LM2576T-ADJ, U3 MCP3428, U4 INA169

Commit message: Some work on PCB
Parts:
- added R16: 0R1, Resistors_SMD:R_2512, B.Cu at (141.0, 38.7)
- added R17: 0R1, Resistors_SMD:R_2512, B.Cu at (128.3, 38.7)
- added R18: 0R1, Resistors_SMD:R_2512, B.Cu at (159.4, 43.2)
- added R19: 0R1, Resistors_SMD:R_2512, B.Cu at (155.6, 43.2)
- C6, D1, R1, R10, R11, R12, R13, R14, R15, R2, R3, R4, R8, R9, U1, U3, U4: moved to B.Cu
- moved L2 99.8 mm to (161.9, 36.2), turned to 90 degrees
- moved R7 91.7 mm to (150.5, 19.1)
- moved R6 90.8 mm to (149.9, 21.0), turned to 180 degrees
- moved U1 79.9 mm to (133.3, 38.7)
- moved U4 75.2 mm to (167.6, 42.5), turned to 180 degrees
- moved R5 73.7 mm to (144.8, 28.6)
- moved Q1 69.5 mm to (149.9, 28.6), turned to 180 degrees
- moved R4 68.0 mm to (132.7, 42.5), turned to 180 degrees
- moved J2 66.1 mm to (155.6, 48.9)
- moved R12 65.8 mm to (151.8, 43.8), turned to 180 degrees
- moved U3 65.6 mm to (145.4, 51.4), turned to 180 degrees
- moved J1 65.2 mm to (132.1, 51.4), turned to 180 degrees
- moved R2 61.6 mm to (135.9, 48.9), turned to 270 degrees
- moved R1 61.6 mm to (135.9, 45.7), turned to 270 degrees
- moved R13 59.8 mm to (151.1, 47.0), turned to 270 degrees
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Connections:
- U3 pad 1: IN_Voltage -> OUT_Voltage
- U3 pad 11: OUT_Voltage -> IN_Voltage
- U3 pad 13: OUT_Current -> IN_Current
- U3 pad 3: IN_Current -> OUT_Current
Routing:
- net GNDA: track 0.00 -> 52.3 mm
- net Net-(C2-Pad1): track 0.00 -> 40.9 mm
- net Net-(D1-Pad1): track 0.00 -> 28.5 mm
- net Net-(C4-Pad1): track 0.00 -> 14.1 mm
- net Net-(C1-Pad1): track 0.00 -> 9.31 mm
- net Net-(R6-Pad2): track 0.00 -> 5.32 mm
Other:
- net class Default: trace_width 0.25 -> 0.8; via_dia 0.6 -> 1.2; via_drill 0.4 -> 0.8
- net class Power added: clearance 0.2, trace_width 1.6, via_dia 2, via_drill 1.2

Commit message: PCB work
Parts:
- moved R15 16.0 mm to (152.4, 40.0)
- moved C5 7.96 mm to (152.4, 54.0), turned to 90 degrees
- moved C6 6.75 mm to (150.5, 52.7), turned to 90 degrees
- moved R4 6.63 mm to (126.4, 44.5)
- moved U1 6.35 mm to (127.0, 38.7)
- moved J2 5.68 mm to (160.7, 51.4)
- moved R2 2.84 mm to (137.2, 46.4), turned to 0 degrees
- moved J1 2.69 mm to (130.2, 53.3)
- moved R9 2.62 mm to (140.3, 54.0)
- moved R8 2.54 mm to (139.7, 56.5)
- moved R16 2.54 mm to (138.4, 38.7)
- moved R17 2.54 mm to (130.8, 38.7)
- moved R3 2.54 mm to (134.6, 38.7)
- moved U4 2.29 mm to (168.9, 44.5)
- moved R14 2.29 mm to (165.1, 44.5)
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Routing:
- net GNDA: track 52.3 -> 108.5 mm
- net Net-(C1-Pad1): track 9.31 -> 40.7 mm
- net Net-(J1-Pad2): track 0.00 -> 24.7 mm

Commit message: Finishing PCB
Parts:
- J2: footprint Socket_Strips:Socket_Strip_Straight_2x03_Pitch2.54mm -> Pin_Headers:Pin_Header_Straight_2x03_Pitch2.54mm
- R1, R12, R13, R15, R2, R4: moved to F.Cu
- moved R4 16.6 mm to (140.3, 53.3), turned to 0 degrees
- moved R15 13.9 mm to (145.4, 52.1), turned to 270 degrees
- moved J2 7.01 mm to (160.0, 58.4), turned to 180 degrees
- moved R7 6.35 mm to (150.5, 25.4), turned to 270 degrees
- moved R13 6.02 mm to (145.4, 48.9), turned to 180 degrees
- moved R2 5.46 mm to (140.3, 50.8)
- moved R10 5.46 mm to (132.7, 59.7)
- moved R11 5.46 mm to (132.7, 57.1)
- moved R8 5.46 mm to (135.3, 59.7)
- moved J3 5.46 mm to (165.7, 55.9), turned to 180 degrees
- moved R12 5.43 mm to (149.9, 48.9)
- moved R9 5.12 mm to (135.9, 56.5)
- moved R6 4.49 mm to (153.0, 24.1)
- moved R1 4.07 mm to (137.8, 48.3)
- moved C5 3.17 mm to (149.9, 55.9)
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Connections:
- U3 pad 11: IN_Voltage -> IN_Current
- U3 pad 13: IN_Current -> IN_Voltage
Routing:
- net GNDA: track 108.5 -> 219.6 mm
- net Net-(C4-Pad1): track 14.1 -> 51.8 mm, vias 0 -> 1
- net OUT_Current: track 0.00 -> 33.3 mm, vias 0 -> 2
- net SCL: track 0.00 -> 33.1 mm, vias 0 -> 2
- net PowerEnable: track 0.00 -> 28.4 mm, vias 0 -> 1
- net Net-(J3-Pad2): track 0.00 -> 20.9 mm
- net +5V: track 0.00 -> 15.0 mm
- net SDA: track 0.00 -> 13.0 mm
- net Net-(J1-Pad2): track 24.7 -> 31.4 mm, vias 0 -> 1
- net Net-(Q1-Pad3): track 0.00 -> 6.31 mm
- net OUT_Voltage: track 0.00 -> 5.82 mm, vias 0 -> 1
- net IN_Voltage: track 0.00 -> 4.55 mm, vias 0 -> 1
- net Net-(C1-Pad1): track 40.7 -> 44.7 mm
- net Net-(C2-Pad1): track 40.9 -> 36.9 mm
- net Net-(R6-Pad2): track 5.32 -> 7.02 mm
Other:
- net class Default: clearance 0.2 -> 0.2032; trace_width 0.8 -> 0.8128; via_dia 1.2 -> 1.4
- net class Power: clearance 0.2 -> 0.2032; trace_width 1.6 -> 1.6256
- rule trace_clearance: 0.2 -> 0.2032

Commit message: Finishing PCB
Parts:
- added C7: 100n, Capacitors_SMD:C_0805, B.Cu at (124.5, 36.2)
- added C8: 100n, Capacitors_SMD:C_0805, B.Cu at (170.8, 47.0)
- added REF**: MountingHole_3.2mm_M3_Pad, Mounting_Holes:MountingHole_3.2mm_M3_Pad, F.Cu at (122.6, 56.5)
- added REF**: MountingHole_3.2mm_M3_Pad, Mounting_Holes:MountingHole_3.2mm_M3_Pad, F.Cu at (174.6, 56.5)
- added REF**: MountingHole_3.2mm_M3_Pad, Mounting_Holes:MountingHole_3.2mm_M3_Pad, F.Cu at (174.6, 20.3)
- added REF**: MountingHole_3.2mm_M3_Pad, Mounting_Holes:MountingHole_3.2mm_M3_Pad, F.Cu at (122.6, 20.3)
- R15, R4: moved to B.Cu
- moved R15 26.8 mm to (170.2, 41.9), turned to 0 degrees
- moved R4 19.4 mm to (125.1, 41.3), turned to 180 degrees
- moved R8 4.45 mm to (135.3, 55.2), turned to 0 degrees
- moved R10 3.59 mm to (135.3, 57.1), turned to 0 degrees
- moved R9 3.24 mm to (135.3, 53.3), turned to 180 degrees
- moved R11 3.17 mm to (135.3, 59.1), turned to 180 degrees
- moved R1 1.27 mm to (137.8, 47.0)
Routing:
- net IN_Current: track 0.00 -> 22.7 mm, vias 0 -> 2
- net +5V: track 15.0 -> 36.1 mm, vias 0 -> 1
- net GNDA: track 219.6 -> 231.6 mm
- net Net-(R10-Pad2): track 0.00 -> 6.40 mm
- net Net-(R8-Pad2): track 0.00 -> 6.14 mm
- net IN_Voltage: track 4.55 -> 6.72 mm
- net Net-(C4-Pad1): track 51.8 -> 53.8 mm
- net Net-(C7-Pad2): track 31.4 -> 32.1 mm
- net SCL: track 33.1 -> 32.6 mm
Other:
- board outline added: 61 x 47 mm
- board text added: "IN"
- board text added: "OUT"
- board text added: "PowerSupply JP, 7.12.2017"
