File: Power Supply LM2576/Power Supply LM2576.sch (KiCad schematic (older format))
At the start: 36 parts, among them J1 Power IN, J2 Conn_02x03_Odd_Even, J3 Power OUT, Q1 IRLML0030, U1 INA169, U2 LM2576T-ADJ, U3 MCP3428, U4 INA169

Commit message: Finishing PCB
Parts:
- J2: footprint Socket_Strips:Socket_Strip_Straight_2x03_Pitch2.54mm -> Pin_Headers:Pin_Header_Straight_2x03_Pitch2.54mm
Connections:
- net IN_Current: now also U3.11 (CH3+); no longer U3.13 (CH4+)
- net IN_Voltage: now also U3.13 (CH4+); no longer U3.11 (CH3+)
Changed lines of the file:
@@
 $EndComp
 $Comp
-L GNDA #PWR10
+L GNDA #PWR01
 U 1 1 59FFC0A0
 P 5050 4200
-F 0 "#PWR10" H 5050 3950 50  0001 C CNN
+F 0 "#PWR01" H 5050 3950 50  0001 C CNN
 F 1 "GNDA" H 5050 4050 50  0000 C CNN
 F 2 "" H 5050 4200 50  0001 C CNN
@@
 $EndComp
 $Comp
-L GNDA #PWR19
+L GNDA #PWR02
 U 1 1 59FFC329
 P 6550 4200
-F 0 "#PWR19" H 6550 3950 50  0001 C CNN
+F 0 "#PWR02" H 6550 3950 50  0001 C CNN
 F 1 "GNDA" H 6550 4050 50  0000 C CNN
 F 2 "" H 6550 4200 50  0001 C CNN
@@
 $EndComp
 $Comp
-L GNDA #PWR18
+L GNDA #PWR03
 U 1 1 59FFC346
 P 6250 4600
-F 0 "#PWR18" H 6250 4350 50  0001 C CNN
+F 0 "#PWR03" H 6250 4350 50  0001 C CNN
 F 1 "GNDA" H 6250 4450 50  0000 C CNN
 F 2 "" H 6250 4600 50  0001 C CNN
@@
 $EndComp
 $Comp
-L GNDA #PWR4
+L GNDA #PWR04
 U 1 1 59FFC406
 P 3750 4200
-F 0 "#PWR4" H 3750 3950 50  0001 C CNN
+F 0 "#PWR04" H 3750 3950 50  0001 C CNN
 F 1 "GNDA" H 3750 4050 50  0000 C CNN
 F 2 "" H 3750 4200 50  0001 C CNN
@@
 $EndComp
 $Comp
-L GNDA #PWR2
+L GNDA #PWR05
 U 1 1 59FFC542
 P 3050 3800
-F 0 "#PWR2" H 3050 3550 50  0001 C CNN
+F 0 "#PWR05" H 3050 3550 50  0001 C CNN
 F 1 "GNDA" H 3050 3650 50  0000 C CNN
 F 2 "" H 3050 3800 50  0001 C CNN
@@
 $EndComp
 $Comp
-L GNDA #PWR31
+L GNDA #PWR06
 U 1 1 59FFC652
 P 8000 4000
-F 0 "#PWR31" H 8000 3750 50  0001 C CNN
+F 0 "#PWR06" H 8000 3750 50  0001 C CNN
 F 1 "GNDA" H 8000 3850 50  0000 C CNN
 F 2 "" H 8000 4000 50  0001 C CNN
@@
 $EndComp
 $Comp
-L GNDA #PWR11
+L GNDA #PWR07
 U 1 1 59FFC8D5
 P 5650 4200
-F 0 "#PWR11" H 5650 3950 50  0001 C CNN
+F 0 "#PWR07" H 5650 3950 50  0001 C CNN
 F 1 "GNDA" H 5650 4050 50  0000 C CNN
 F 2 "" H 5650 4200 50  0001 C CNN
@@
 $EndComp
 $Comp
-L GNDA #PWR9
+L GNDA #PWR08
 U 1 1 5A0254E4
 P 4350 4700
-F 0 "#PWR9" H 4350 4450 50  0001 C CNN
+F 0 "#PWR08" H 4350 4450 50  0001 C CNN
 F 1 "GNDA" H 4350 4550 50  0000 C CNN
 F 2 "" H 4350 4700 50  0001 C CNN
@@
 $EndComp
 $Comp
-L GNDA #PWR20
+L GNDA #PWR09
 U 1 1 5A025A22
 P 6850 4200
-F 0 "#PWR20" H 6850 3950 50  0001 C CNN
+F 0 "#PWR09" H 6850 3950 50  0001 C CNN
 F 1 "GNDA" H 6850 4050 50  0000 C CNN
 F 2 "" H 6850 4200 50  0001 C CNN
@@
 $EndComp
 $Comp
-L GNDA #PWR26
+L GNDA #PWR010
 U 1 1 5A025EC7
 P 7450 4200
-F 0 "#PWR26" H 7450 3950 50  0001 C CNN
+F 0 "#PWR010" H 7450 3950 50  0001 C CNN
 F 1 "GNDA" H 7450 4050 50  0000 C CNN
 F 2 "" H 7450 4200 50  0001 C CNN
@@
 Connection ~ 3600 3650
 $Comp
-L GNDA #PWR5
+L GNDA #PWR011
 U 1 1 5A03B368
 P 4000 2950
-F 0 "#PWR5" H 4000 2700 50  0001 C CNN
+F 0 "#PWR011" H 4000 2700 50  0001 C CNN
 F 1 "GNDA" H 4000 2800 50  0000 C CNN
 F 2 "" H 4000 2950 50  0001 C CNN
@@
 	4350 2600 4350 2650
 $Comp
-L GNDA #PWR8
+L GNDA #PWR012
 U 1 1 5A03B53A
 P 4350 2950
-F 0 "#PWR8" H 4350 2700 50  0001 C CNN
+F 0 "#PWR012" H 4350 2700 50  0001 C CNN
 F 1 "GNDA" H 4350 2800 50  0000 C CNN
 F 2 "" H 4350 2950 50  0001 C CNN
@@
 	7950 2650 8000 2650
 $Comp
-L GNDA #PWR32
+L GNDA #PWR013
 U 1 1 5A03B8EA
 P 8350 2950
-F 0 "#PWR32" H 8350 2700 50  0001 C CNN
+F 0 "#PWR013" H 8350 2700 50  0001 C CNN
 F 1 "GNDA" H 8350 2800 50  0000 C CNN
 F 2 "" H 8350 2950 50  0001 C CNN
@@
 	8700 2600 8700 2650
 $Comp
-L GNDA #PWR33
+L GNDA #PWR014
 U 1 1 5A03B8F8
 P 8700 2950
-F 0 "#PWR33" H 8700 2700 50  0001 C CNN
+F 0 "#PWR014" H 8700 2700 50  0001 C CNN
 F 1 "GNDA" H 8700 2800 50  0000 C CNN
 F 2 "" H 8700 2950 50  0001 C CNN
@@
 $EndComp
 $Comp
-L +5V #PWR27
+L +5V #PWR015
 U 1 1 5A03C42C
 P 7500 1350
-F 0 "#PWR27" H 7500 1200 50  0001 C CNN
+F 0 "#PWR015" H 7500 1200 50  0001 C CNN
 F 1 "+5V" H 7500 1490 50  0000 C CNN
 F 2 "" H 7500 1350 50  0001 C CNN
@@
 $EndComp
 $Comp
-L +5V #PWR29
+L +5V #PWR016
 U 1 1 5A03C4F6
 P 7800 1350
-F 0 "#PWR29" H 7800 1200 50  0001 C CNN
+F 0 "#PWR016" H 7800 1200 50  0001 C CNN
 F 1 "+5V" H 7800 1490 50  0000 C CNN
 F 2 "" H 7800 1350 50  0001 C CNN
@@
 $EndComp
 $Comp
-L +5V #PWR16
+L +5V #PWR017
 U 1 1 5A03C65A
 P 6150 1100
-F 0 "#PWR16" H 6150 950 50  0001 C CNN
+F 0 "#PWR017" H 6150 950 50  0001 C CNN
 F 1 "+5V" H 6150 1240 50  0000 C CNN
 F 2 "" H 6150 1100 50  0001 C CNN
@@
 $EndComp
 $Comp
-L GNDA #PWR30
+L GNDA #PWR018
 U 1 1 5A03CBEF
 P 7800 1650
-F 0 "#PWR30" H 7800 1400 50  0001 C CNN
+F 0 "#PWR018" H 7800 1400 50  0001 C CNN
 F 1 "GNDA" H 7800 1500 50  0000 C CNN
 F 2 "" H 7800 1650 50  0001 C CNN
@@
 $EndComp
 $Comp
-L GNDA #PWR28
+L GNDA #PWR019
 U 1 1 5A03CC3F
 P 7500 1650
-F 0 "#PWR28" H 7500 1400 50  0001 C CNN
+F 0 "#PWR019" H 7500 1400 50  0001 C CNN
 F 1 "GNDA" H 7500 1500 50  0000 C CNN
 F 2 "" H 7500 1650 50  0001 C CNN
@@
 $EndComp
 $Comp
-L GNDA #PWR17
+L GNDA #PWR020
 U 1 1 5A03CC8F
 P 6150 2200
-F 0 "#PWR17" H 6150 1950 50  0001 C CNN
+F 0 "#PWR020" H 6150 1950 50  0001 C CNN
 F 1 "GNDA" H 6150 2050 50  0000 C CNN
 F 2 "" H 6150 2200 50  0001 C CNN
@@
 $EndComp
 $Comp
-L GNDA #PWR12
+L GNDA #PWR021
 U 1 1 5A03CD97
 P 5750 1400
-F 0 "#PWR12" H 5750 1150 50  0001 C CNN
+F 0 "#PWR021" H 5750 1150 50  0001 C CNN
 F 1 "GNDA" H 5750 1250 50  0000 C CNN
 F 2 "" H 5750 1400 50  0001 C CNN
@@
 $EndComp
 $Comp
-L GNDA #PWR13
+L GNDA #PWR022
 U 1 1 5A03CE34
 P 5750 1600
-F 0 "#PWR13" H 5750 1350 50  0001 C CNN
+F 0 "#PWR022" H 5750 1350 50  0001 C CNN
 F 1 "GNDA" H 5750 1450 50  0000 C CNN
 F 2 "" H 5750 1600 50  0001 C CNN
@@
 $EndComp
 $Comp
-L GNDA #PWR14
+L GNDA #PWR023
 U 1 1 5A03CE84
 P 5750 1800
-F 0 "#PWR14" H 5750 1550 50  0001 C CNN
+F 0 "#PWR023" H 5750 1550 50  0001 C CNN
 F 1 "GNDA" H 5750 1650 50  0000 C CNN
 F 2 "" H 5750 1800 50  0001 C CNN
@@
 $EndComp
 $Comp
-L GNDA #PWR15
+L GNDA #PWR024
 U 1 1 5A03CED4
 P 5750 2000
-F 0 "#PWR15" H 5750 1750 50  0001 C CNN
+F 0 "#PWR024" H 5750 1750 50  0001 C CNN
 F 1 "GNDA" H 5750 1850 50  0000 C CNN
 F 2 "" H 5750 2000 50  0001 C CNN
@@
 OUT_Current
 Connection ~ 8700 2600
-Text GLabel 5450 1900 0    60   Input ~ 0
+Text GLabel 5450 1700 0    60   Input ~ 0
 IN_Current
 Text GLabel 5450 1500 0    60   Input ~ 0
@@
 $EndComp
 $Comp
-L GNDA #PWR1
+L GNDA #PWR025
 U 1 1 5A03E32E
 P 2950 3300
-F 0 "#PWR1" H 2950 3050 50  0001 C CNN
+F 0 "#PWR025" H 2950 3050 50  0001 C CNN
 F 1 "GNDA" H 2950 3150 50  0000 C CNN
 F 2 "" H 2950 3300 50  0001 C CNN
@@
 $EndComp
 $Comp
-L GNDA #PWR25
+L GNDA #PWR026
 U 1 1 5A03E84E
 P 7350 3300
-F 0 "#PWR25" H 7350 3050 50  0001 C CNN
+F 0 "#PWR026" H 7350 3050 50  0001 C CNN
 F 1 "GNDA" H 7350 3150 50  0000 C CNN
 F 2 "" H 7350 3300 50  0001 C CNN
@@
 Text GLabel 5450 1300 0    60   Input ~ 0
 OUT_Voltage
-Text GLabel 5450 1700 0    60   Input ~ 0
+Text GLabel 5450 1900 0    60   Input ~ 0
 IN_Voltage
 Wire Wire Line
@@
 Connection ~ 7050 1700
 $Comp
-L GNDA #PWR22
+L GNDA #PWR027
 U 1 1 5A03F4A2
 P 7050 2150
-F 0 "#PWR22" H 7050 1900 50  0001 C CNN
+F 0 "#PWR027" H 7050 1900 50  0001 C CNN
 F 1 "GNDA" H 7050 2000 50  0000 C CNN
 F 2 "" H 7050 2150 50  0001 C CNN
@@
 $EndComp
 $Comp
-L +5V #PWR21
+L +5V #PWR028
 U 1 1 5A03F504
 P 7050 1350
-F 0 "#PWR21" H 7050 1200 50  0001 C CNN
+F 0 "#PWR028" H 7050 1200 50  0001 C CNN
 F 1 "+5V" H 7050 1490 50  0000 C CNN
 F 2 "" H 7050 1350 50  0001 C CNN
@@
 Connection ~ 7250 1800
 $Comp
-L GNDA #PWR24
+L GNDA #PWR029
 U 1 1 5A03F5DF
 P 7250 2150
-F 0 "#PWR24" H 7250 1900 50  0001 C CNN
+F 0 "#PWR029" H 7250 1900 50  0001 C CNN
 F 1 "GNDA" H 7250 2000 50  0000 C CNN
 F 2 "" H 7250 2150 50  0001 C CNN
@@
 $EndComp
 $Comp
-L +5V #PWR23
+L +5V #PWR030
 U 1 1 5A03F5E5
 P 7250 1350
-F 0 "#PWR23" H 7250 1200 50  0001 C CNN
+F 0 "#PWR030" H 7250 1200 50  0001 C CNN
 F 1 "+5V" H 7250 1490 50  0000 C CNN
 F 2 "" H 7250 1350 50  0001 C CNN
@@
 F 0 "J2" H 3800 1750 50  0000 C CNN
 F 1 "Conn_02x03_Odd_Even" H 3800 1350 50  0000 C CNN
-F 2 "Socket_Strips:Socket_Strip_Straight_2x03_Pitch2.54mm" H 3750 1550 50  0001 C CNN
+F 2 "Pin_Headers:Pin_Header_Straight_2x03_Pitch2.54mm" H 3750 1550 50  0001 C CNN
 F 3 "" H 3750 1550 50  0001 C CNN
 	1    3750 1550
@@
 $EndComp
 $Comp
-L GNDA #PWR3
+L GNDA #PWR031
 U 1 1 5A03FA4A
 P 3550 1450
-F 0 "#PWR3" H 3550 1200 50  0001 C CNN
+F 0 "#PWR031" H 3550 1200 50  0001 C CNN
 F 1 "GNDA" H 3550 1300 50  0000 C CNN
 F 2 "" H 3550 1450 50  0001 C CNN
@@
 $EndComp
 $Comp
-L +5V #PWR7
+L +5V #PWR032
 U 1 1 5A03FAB5
 P 4050 1650
-F 0 "#PWR7" H 4050 1500 50  0001 C CNN
+F 0 "#PWR032" H 4050 1500 50  0001 C CNN
 F 1 "+5V" H 4050 1790 50  0000 C CNN
 F 2 "" H 4050 1650 50  0001 C CNN
@@
 $EndComp
 $Comp
-L GNDA #PWR6
+L GNDA #PWR033
 U 1 1 5A03FDB0
 P 4050 1450
-F 0 "#PWR6" H 4050 1200 50  0001 C CNN
+F 0 "#PWR033" H 4050 1200 50  0001 C CNN
 F 1 "GNDA" H 4050 1300 50  0000 C CNN
 F 2 "" H 4050 1450 50  0001 C CNN

Commit message: Finishing PCB
Parts:
- added C7, C8: 100n, Capacitors_SMD:C_0805, symbol C
Connections:
- net GNDA: now also C7.1, C8.1
- net at J1.2 (Pin_2), R1.1, R16.2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: now also C7.2
- net at C4.1, L2.2, R12.1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: now also C8.2
Changed lines of the file:
@@
 Connection ~ 3200 3650
 Wire Wire Line
-	3600 3650 3600 2650
+	3600 2650 3600 3650
 Wire Wire Line
 	3600 2650 3650 2650
@@
 	4000 2350 4000 2300
 Wire Wire Line
-	4000 2300 3200 2300
+	3200 2300 4100 2300
 Connection ~ 3200 2550
 $Comp
@@
 	7900 3850 8050 3850
 Wire Wire Line
-	7950 3850 7950 2650
+	7950 2650 7950 3850
 Wire Wire Line
 	7950 2650 8000 2650
@@
 	8350 2350 8350 2300
 Wire Wire Line
-	8350 2300 7550 2300
+	7550 2300 8450 2300
 Connection ~ 7550 2550
 $Comp
@@
 	7900 3650 7950 3650
 Connection ~ 7950 3650
+$Comp
+L C C7
+U 1 1 5A29D3C5
+P 4250 2300
+F 0 "C7" H 4275 2400 50  0000 L CNN
+F 1 "100n" H 4275 2200 50  0000 L CNN
+F 2 "Capacitors_SMD:C_0805" H 4288 2150 50  0001 C CNN
+F 3 "" H 4250 2300 50  0001 C CNN
+	1    4250 2300
+	0    1    1    0
+$EndComp
+$Comp
+L GNDA #PWR034
+U 1 1 5A29D52D
+P 4400 2300
+F 0 "#PWR034" H 4400 2050 50  0001 C CNN
+F 1 "GNDA" H 4400 2150 50  0000 C CNN
+F 2 "" H 4400 2300 50  0001 C CNN
+F 3 "" H 4400 2300 50  0001 C CNN
+	1    4400 2300
+	0    -1   -1   0
+$EndComp
+Connection ~ 4000 2300
+$Comp
+L C C8
+U 1 1 5A29D7C2
+P 8600 2300
+F 0 "C8" H 8625 2400 50  0000 L CNN
+F 1 "100n" H 8625 2200 50  0000 L CNN
+F 2 "Capacitors_SMD:C_0805" H 8638 2150 50  0001 C CNN
+F 3 "" H 8600 2300 50  0001 C CNN
+	1    8600 2300
+	0    1    1    0
+$EndComp
+$Comp
+L GNDA #PWR035
+U 1 1 5A29D7C8
+P 8750 2300
+F 0 "#PWR035" H 8750 2050 50  0001 C CNN
+F 1 "GNDA" H 8750 2150 50  0000 C CNN
+F 2 "" H 8750 2300 50  0001 C CNN
+F 3 "" H 8750 2300 50  0001 C CNN
+	1    8750 2300
+	0    -1   -1   0
+$EndComp
+Connection ~ 8350 2300
 $EndSCHEMATC
