File: KiCad/Power Supply LMZ14203H/Power Supply LMZ14203H.sch (KiCad schematic (older format))
At the start: 63 parts, among them J1 Power IN, J3 Power OUT, J4 OLED I2C, J5 PDI, J6 OLED, SW1 SW_DIP_x01, U1 INA169, U2 LMZ14203H, U3 L78M12, U4 INA169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

Commit message: Wirering done
Parts:
- J4: footprint Pin_Headers:Pin_Header_Straight_1x04_Pitch2.54mm -> JPDisplays:OLED_0.96inch_128x64_I2C
Connections:
- net GND: now also C7.1, C8.1, R13.2, R15.2, R2.2, R4.2, U1.2 (GND), U4.2 (GND)
- net GNDA: no longer C7.1, C8.1, R13.2, R15.2, R2.2, R4.2, U1.2 (GND), U4.2 (GND)
- net +3.3VA: now reaches C20.1, C21.1, L1.2, U6.32 (AVCC)
Changed lines of the file:
@@
 Connection ~ 4600 2200
-$Comp
-L power:GNDA #PWR03
-U 1 1 5A03B368
-P 5000 1500
-F 0 "#PWR03" H 5000 1250 50  0001 C CNN
-F 1 "GNDA" H 5000 1350 50  0000 C CNN
-F 2 "" H 5000 1500 50  0001 C CNN
-F 3 "" H 5000 1500 50  0001 C CNN
-	1    5000 1500
-	1    0    0    -1
-$EndComp
 $Comp
 L Device:R R4
@@
 Wire Wire Line
 	5350 1150 5350 1200
-$Comp
-L power:GNDA #PWR04
-U 1 1 5A03B53A
-P 5350 1500
-F 0 "#PWR04" H 5350 1250 50  0001 C CNN
-F 1 "GNDA" H 5350 1350 50  0000 C CNN
-F 2 "" H 5350 1500 50  0001 C CNN
-F 3 "" H 5350 1500 50  0001 C CNN
-	1    5350 1500
-	1    0    0    -1
-$EndComp
 Wire Wire Line
 	5000 1500 5000 1400
@@
 	8950 1200 9000 1200
 $Comp
-L power:GNDA #PWR05
-U 1 1 5A03B8EA
-P 9350 1500
-F 0 "#PWR05" H 9350 1250 50  0001 C CNN
-F 1 "GNDA" H 9350 1350 50  0000 C CNN
-F 2 "" H 9350 1500 50  0001 C CNN
-F 3 "" H 9350 1500 50  0001 C CNN
-	1    9350 1500
-	1    0    0    -1
-$EndComp
-$Comp
 L Device:R R15
 U 1 1 5A03B8F0
@@
 Wire Wire Line
 	9700 1150 9700 1200
-$Comp
-L power:GNDA #PWR06
-U 1 1 5A03B8F8
-P 9700 1500
-F 0 "#PWR06" H 9700 1250 50  0001 C CNN
-F 1 "GNDA" H 9700 1350 50  0000 C CNN
-F 2 "" H 9700 1500 50  0001 C CNN
-F 3 "" H 9700 1500 50  0001 C CNN
-	1    9700 1500
-	1    0    0    -1
-$EndComp
 Wire Wire Line
 	9350 1500 9350 1400
@@
 	1    0    0    -1
 $EndComp
-$Comp
-L power:GNDA #PWR07
-U 1 1 5A03E32E
-P 3950 1850
-F 0 "#PWR07" H 3950 1600 50  0001 C CNN
-F 1 "GNDA" H 3950 1700 50  0000 C CNN
-F 2 "" H 3950 1850 50  0001 C CNN
-F 3 "" H 3950 1850 50  0001 C CNN
-	1    3950 1850
-	1    0    0    -1
-$EndComp
 Wire Wire Line
 	3950 1450 3950 1500
@@
 F 3 "" H 8350 1700 50  0001 C CNN
 	1    8350 1700
-	1    0    0    -1
-$EndComp
-$Comp
-L power:GNDA #PWR08
-U 1 1 5A03E84E
-P 8350 1850
-F 0 "#PWR08" H 8350 1600 50  0001 C CNN
-F 1 "GNDA" H 8350 1700 50  0000 C CNN
-F 2 "" H 8350 1850 50  0001 C CNN
-F 3 "" H 8350 1850 50  0001 C CNN
-	1    8350 1850
 	1    0    0    -1
 $EndComp
@@
 	0    1    1    0
 $EndComp
-$Comp
-L power:GNDA #PWR09
-U 1 1 5A29D52D
-P 5400 850
-F 0 "#PWR09" H 5400 600 50  0001 C CNN
-F 1 "GNDA" H 5400 700 50  0000 C CNN
-F 2 "" H 5400 850 50  0001 C CNN
-F 3 "" H 5400 850 50  0001 C CNN
-	1    5400 850
-	0    -1   -1   0
-$EndComp
 Connection ~ 5000 850
 $Comp
@@
 	1    9600 850
 	0    1    1    0
-$EndComp
-$Comp
-L power:GNDA #PWR010
-U 1 1 5A29D7C8
-P 9750 850
-F 0 "#PWR010" H 9750 600 50  0001 C CNN
-F 1 "GNDA" H 9750 700 50  0000 C CNN
-F 2 "" H 9750 850 50  0001 C CNN
-F 3 "" H 9750 850 50  0001 C CNN
-	1    9750 850
-	0    -1   -1   0
 $EndComp
 Connection ~ 9350 850
@@
 F 0 "J4" H 1300 5800 50  0000 C CNN
 F 1 "OLED I2C" H 1300 5300 50  0000 C CNN
-F 2 "Pin_Headers:Pin_Header_Straight_1x04_Pitch2.54mm" H 1300 5600 50  0001 C CNN
+F 2 "JPDisplays:OLED_0.96inch_128x64_I2C" H 1300 5600 50  0001 C CNN
 F 3 "" H 1300 5600 50  0001 C CNN
 	1    1300 5600
@@
 Wire Wire Line
 	2500 3100 2900 3100
+Text Label 5100 4200 0    50   ~ 0
++3.3VA
+$Comp
+L power:GND #PWR0101
+U 1 1 5B762C27
+P 3950 1850
+F 0 "#PWR0101" H 3950 1600 50  0001 C CNN
+F 1 "GND" H 3950 1700 50  0000 C CNN
+F 2 "" H 3950 1850 50  0001 C CNN
+F 3 "" H 3950 1850 50  0001 C CNN
+	1    3950 1850
+	1    0    0    -1
+$EndComp
+$Comp
+L power:GND #PWR0102
+U 1 1 5B762CB0
+P 5000 1500
+F 0 "#PWR0102" H 5000 1250 50  0001 C CNN
+F 1 "GND" H 5000 1350 50  0000 C CNN
+F 2 "" H 5000 1500 50  0001 C CNN
+F 3 "" H 5000 1500 50  0001 C CNN
+	1    5000 1500
+	1    0    0    -1
+$EndComp
+$Comp
+L power:GND #PWR0103
+U 1 1 5B762D39
+P 5350 1500
+F 0 "#PWR0103" H 5350 1250 50  0001 C CNN
+F 1 "GND" H 5350 1350 50  0000 C CNN
+F 2 "" H 5350 1500 50  0001 C CNN
+F 3 "" H 5350 1500 50  0001 C CNN
+	1    5350 1500
+	1    0    0    -1
+$EndComp
+$Comp
+L power:GND #PWR0104
+U 1 1 5B76307A
+P 9350 1500
+F 0 "#PWR0104" H 9350 1250 50  0001 C CNN
+F 1 "GND" H 9350 1350 50  0000 C CNN
+F 2 "" H 9350 1500 50  0001 C CNN
+F 3 "" H 9350 1500 50  0001 C CNN
+	1    9350 1500
+	1    0    0    -1
+$EndComp
+$Comp
+L power:GND #PWR0105
+U 1 1 5B763103
+P 9700 1500
+F 0 "#PWR0105" H 9700 1250 50  0001 C CNN
+F 1 "GND" H 9700 1350 50  0000 C CNN
+F 2 "" H 9700 1500 50  0001 C CNN
+F 3 "" H 9700 1500 50  0001 C CNN
+	1    9700 1500
+	1    0    0    -1
+$EndComp
+$Comp
+L power:GND #PWR0106
+U 1 1 5B76318C
+P 8350 1850
+F 0 "#PWR0106" H 8350 1600 50  0001 C CNN
+F 1 "GND" H 8350 1700 50  0000 C CNN
+F 2 "" H 8350 1850 50  0001 C CNN
+F 3 "" H 8350 1850 50  0001 C CNN
+	1    8350 1850
+	1    0    0    -1
+$EndComp
+$Comp
+L power:GND #PWR?
+U 1 1 5B763571
+P 5400 850
+F 0 "#PWR?" H 5400 600 50  0001 C CNN
+F 1 "GND" H 5400 700 50  0000 C CNN
+F 2 "" H 5400 850 50  0001 C CNN
+F 3 "" H 5400 850 50  0001 C CNN
+	1    5400 850
+	0    -1   -1   0
+$EndComp
+$Comp
+L power:GND #PWR?
+U 1 1 5B763871
+P 9750 850
+F 0 "#PWR?" H 9750 600 50  0001 C CNN
+F 1 "GND" H 9750 700 50  0000 C CNN
+F 2 "" H 9750 850 50  0001 C CNN
+F 3 "" H 9750 850 50  0001 C CNN
+	1    9750 850
+	0    -1   -1   0
+$EndComp
 $EndSCHEMATC
