File: KiCad/Power Supply LMZ14203H/Power Supply LMZ14203H.sch (KiCad schematic (older format))
At the start: 69 parts, among them J1 Power IN, J3 Power OUT, J4 OLED I2C, J5 PDI, J6 OLED, SW1 SW_DIP_x01, U1 INA169, U2 LMZ14203H, U3 L78M12, U4 INA169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

Commit message: PCB proofing
Parts:
- C10, C9: renamed from C?; footprint Capacitors_Tantalum_SMD:CP_Tantalum_Case-D_EIA-7343-31_Hand -> Capacitors_Tantalum_SMD:CP_Tantalum_Case-D_EIA-7343-31_Reflow
Changed lines of the file:
@@
 	8100 2200 8550 2200
 $Comp
-L Device:CP C?
+L Device:CP C9
 U 1 1 5BF09AEE
 P 7850 2700
-F 0 "C?" H 7875 2800 50  0000 L CNN
+F 0 "C9" H 7875 2800 50  0000 L CNN
 F 1 "47u/1-45mESR" H 7875 2600 50  0000 L CNN
-F 2 "Capacitors_Tantalum_SMD:CP_Tantalum_Case-D_EIA-7343-31_Hand" H 7888 2550 50  0001 C CNN
+F 2 "Capacitors_Tantalum_SMD:CP_Tantalum_Case-D_EIA-7343-31_Reflow" H 7888 2550 50  0001 C CNN
 F 3 "" H 7850 2700 50  0001 C CNN
 	1    7850 2700
@@
 $EndComp
 $Comp
-L Device:CP C?
+L Device:CP C10
 U 1 1 5BF0A518
 P 8100 2700
-F 0 "C?" H 8125 2800 50  0000 L CNN
+F 0 "C10" H 8125 2800 50  0000 L CNN
 F 1 "47u/1-45mESR" H 8125 2600 50  0000 L CNN
-F 2 "Capacitors_Tantalum_SMD:CP_Tantalum_Case-D_EIA-7343-31_Hand" H 8138 2550 50  0001 C CNN
+F 2 "Capacitors_Tantalum_SMD:CP_Tantalum_Case-D_EIA-7343-31_Reflow" H 8138 2550 50  0001 C CNN
 F 3 "" H 8100 2700 50  0001 C CNN
 	1    8100 2700

Commit message: Software init commit
Parts:
- C25, C27: value 100n -> 1u
- L1: footprint Inductors_SMD:L_0805 -> Inductors_SMD:L_1206
- R1: value 90k -> 68k
- R15, R4: value 10k -> 20k
- R2: value 10k -> 2k2
Connections:
- wire segments 232 -> 233
Changed lines of the file:
@@
 P 5350 1350
 F 0 "R4" V 5430 1350 50  0000 C CNN
-F 1 "10k" V 5350 1350 50  0000 C CNN
+F 1 "20k" V 5350 1350 50  0000 C CNN
 F 2 "Resistors_SMD:R_0805" V 5280 1350 50  0001 C CNN
 F 3 "" H 5350 1350 50  0001 C CNN
@@
 P 9700 1350
 F 0 "R15" V 9780 1350 50  0000 C CNN
-F 1 "10k" V 9700 1350 50  0000 C CNN
+F 1 "20k" V 9700 1350 50  0000 C CNN
 F 2 "Resistors_SMD:R_0805" V 9630 1350 50  0001 C CNN
 F 3 "" H 9700 1350 50  0001 C CNN
@@
 P 3950 1300
 F 0 "R1" V 4030 1300 50  0000 C CNN
-F 1 "90k" V 3950 1300 50  0000 C CNN
+F 1 "68k" V 3950 1300 50  0000 C CNN
 F 2 "Resistors_SMD:R_0805" V 3880 1300 50  0001 C CNN
 F 3 "" H 3950 1300 50  0001 C CNN
@@
 P 3950 1700
 F 0 "R2" V 4030 1700 50  0000 C CNN
-F 1 "10k" V 3950 1700 50  0000 C CNN
+F 1 "2k2" V 3950 1700 50  0000 C CNN
 F 2 "Resistors_SMD:R_0805" V 3880 1700 50  0001 C CNN
 F 3 "" H 3950 1700 50  0001 C CNN
@@
 F 0 "L1" V 4900 4200 50  0000 C CNN
 F 1 "10u" V 5025 4200 50  0000 C CNN
-F 2 "Inductors_SMD:L_0805" H 4950 4200 50  0001 C CNN
+F 2 "Inductors_SMD:L_1206" H 4950 4200 50  0001 C CNN
 F 3 "" H 4950 4200 50  0001 C CNN
 	1    4950 4200
@@
 	1    0    0    -1
 $EndComp
+Text GLabel 1250 4650 0    60   Input ~ 0
+PDI_CLK
 Text GLabel 1250 4450 0    60   Input ~ 0
-PDI_CLK
-Text GLabel 1250 4650 0    60   Input ~ 0
 PDI_DATA
 $Comp
@@
 P 5500 1350
 F 0 "C25" H 5525 1450 50  0000 L CNN
-F 1 "100n" H 5525 1250 50  0000 L CNN
+F 1 "1u" H 5525 1250 50  0000 L CNN
 F 2 "Capacitors_SMD:C_0805" H 5538 1200 50  0001 C CNN
 F 3 "" H 5500 1350 50  0001 C CNN
@@
 P 9850 1350
 F 0 "C27" H 9875 1450 50  0000 L CNN
-F 1 "100n" H 9875 1250 50  0000 L CNN
+F 1 "1u" H 9875 1250 50  0000 L CNN
 F 2 "Capacitors_SMD:C_0805" H 9888 1200 50  0001 C CNN
 F 3 "" H 9850 1350 50  0001 C CNN
@@
 Wire Wire Line
 	3700 2150 3700 2200
-Wire Bus Line
-	2850 6200 2850 7050
-Wire Bus Line
-	6750 5350 6750 7050
-Wire Bus Line
-	9500 3700 9500 5350
 Connection ~ 3700 2200
 Wire Wire Line
@@
 	1    0    0    -1
 $EndComp
+$Comp
+L power:+3.3V #PWR0113
+U 1 1 5BA87682
+P 9850 5100
+F 0 "#PWR0113" H 9850 4950 50  0001 C CNN
+F 1 "+3.3V" H 9850 5240 50  0000 C CNN
+F 2 "" H 9850 5100 50  0001 C CNN
+F 3 "" H 9850 5100 50  0001 C CNN
+	1    9850 5100
+	1    0    0    -1
+$EndComp
+Wire Wire Line
+	9850 5100 9850 5200
+Connection ~ 9850 5200
+Wire Bus Line
+	2850 6200 2850 7050
+Wire Bus Line
+	6750 5350 6750 7050
+Wire Bus Line
+	9500 3700 9500 5350
 $EndSCHEMATC

Commit message: Screen.cpp added, some clean up, too
Parts:
- C12: value 10n -> 220n
Changed lines of the file:
@@
 P 1800 7000
 F 0 "C12" H 1825 7100 50  0000 L CNN
-F 1 "10n" H 1825 6900 50  0000 L CNN
+F 1 "220n" H 1825 6900 50  0000 L CNN
 F 2 "Capacitors_SMD:C_0805" H 1838 6850 50  0001 C CNN
 F 3 "" H 1800 7000 50  0001 C CNN

Commit message: MobilePowerBank ADC first code
Parts:
- added D?: 1N4007, Diode_THT:D_DO-41_SOD81_P10.16mm_Horizontal, symbol Diode:1N4007
- added Q?: BC548, Package_TO_SOT_THT:TO-92_Inline, symbol Transistor_BJT:BC548
- added R? (x2): 47k, Resistors_SMD:R_0805, symbol Device:R
- added R?: 4k7, Resistors_SMD:R_0805, symbol Device:R
Connections:
- net labels added: PowerSense
- wire segments 233 -> 241
Other:
- note added: "VinMax = 35V"
Changed lines of the file:
@@
 Wire Wire Line
 	4650 3200 4650 3300
-Text GLabel 1200 3000 1    60   Input ~ 0
+Text GLabel 1200 2550 1    60   Input ~ 0
 POWER_IN
 Connection ~ 1200 3100
@@
 	9850 5100 9850 5200
 Connection ~ 9850 5200
+Text Notes 550  2350 0    50   ~ 0
+VinMax = 35V
+$Comp
+L Diode:1N4007 D?
+U 1 1 5C20097F
+P 1200 2850
+F 0 "D?" V 1246 2771 50  0000 R CNN
+F 1 "1N4007" V 1155 2771 50  0000 R CNN
+F 2 "Diode_THT:D_DO-41_SOD81_P10.16mm_Horizontal" H 1200 2675 50  0001 C CNN
+F 3 "http://www.vishay.com/docs/88503/1n4001.pdf" H 1200 2850 50  0001 C CNN
+	1    1200 2850
+	0    -1   -1   0
+$EndComp
+$Comp
+L power:+3.3V #PWR?
+U 1 1 5C23B876
+P 2300 1300
+F 0 "#PWR?" H 2300 1150 50  0001 C CNN
+F 1 "+3.3V" H 2300 1440 50  0000 C CNN
+F 2 "" H 2300 1300 50  0001 C CNN
+F 3 "" H 2300 1300 50  0001 C CNN
+	1    2300 1300
+	1    0    0    -1
+$EndComp
+Wire Wire Line
+	1200 2550 1200 2700
+Text GLabel 1850 1550 1    60   Input ~ 0
+POWER_IN
+$Comp
+L Device:R R?
+U 1 1 5C2E23E0
+P 1850 1700
+F 0 "R?" V 1930 1700 50  0000 C CNN
+F 1 "47k" V 1850 1700 50  0000 C CNN
+F 2 "Resistors_SMD:R_0805" V 1780 1700 50  0001 C CNN
+F 3 "" H 1850 1700 50  0001 C CNN
+	1    1850 1700
+	1    0    0    -1
+$EndComp
+$Comp
+L Device:R R?
+U 1 1 5C311AF4
+P 1850 2100
+F 0 "R?" V 1930 2100 50  0000 C CNN
+F 1 "4k7" V 1850 2100 50  0000 C CNN
+F 2 "Resistors_SMD:R_0805" V 1780 2100 50  0001 C CNN
+F 3 "" H 1850 2100 50  0001 C CNN
+	1    1850 2100
+	1    0    0    -1
+$EndComp
+$Comp
+L Transistor_BJT:BC548 Q?
+U 1 1 5C311D59
+P 2200 1900
+F 0 "Q?" H 2391 1946 50  0000 L CNN
+F 1 "BC548" H 2391 1855 50  0000 L CNN
+F 2 "Package_TO_SOT_THT:TO-92_Inline" H 2400 1825 50  0001 L CIN
+F 3 "http://www.fairchildsemi.com/ds/BC/BC547.pdf" H 2200 1900 50  0001 L CNN
+	1    2200 1900
+	1    0    0    -1
+$EndComp
+$Comp
+L Device:R R?
+U 1 1 5C311E29
+P 2300 1450
+F 0 "R?" V 2380 1450 50  0000 C CNN
+F 1 "47k" V 2300 1450 50  0000 C CNN
+F 2 "Resistors_SMD:R_0805" V 2230 1450 50  0001 C CNN
+F 3 "" H 2300 1450 50  0001 C CNN
+	1    2300 1450
+	1    0    0    -1
+$EndComp
+$Comp
+L power:GND #PWR?
+U 1 1 5C311EFB
+P 1850 2250
+F 0 "#PWR?" H 1850 2000 50  0001 C CNN
+F 1 "GND" H 1850 2100 50  0000 C CNN
+F 2 "" H 1850 2250 50  0001 C CNN
+F 3 "" H 1850 2250 50  0001 C CNN
+	1    1850 2250
+	1    0    0    -1
+$EndComp
+$Comp
+L power:GND #PWR?
+U 1 1 5C311FA0
+P 2300 2250
+F 0 "#PWR?" H 2300 2000 50  0001 C CNN
+F 1 "GND" H 2300 2100 50  0000 C CNN
+F 2 "" H 2300 2250 50  0001 C CNN
+F 3 "" H 2300 2250 50  0001 C CNN
+	1    2300 2250
+	1    0    0    -1
+$EndComp
+Wire Wire Line
+	2300 2250 2300 2100
+Wire Wire Line
+	1850 1850 1850 1900
+Wire Wire Line
+	1850 1900 2000 1900
+Connection ~ 1850 1900
+Wire Wire Line
+	1850 1900 1850 1950
+Text GLabel 2450 1650 2    50   Input ~ 0
+PowerSense
+Wire Wire Line
+	2450 1650 2300 1650
+Wire Wire Line
+	2300 1600 2300 1650
+Connection ~ 2300 1650
+Wire Wire Line
+	2300 1650 2300 1700
 Wire Bus Line
 	2850 6200 2850 7050
