File: KiCad/Power Supply LMZ14203H/Power Supply LMZ14203H.kicad_pcb (KiCad board)
At the start: 2 copper layers, 92.7 x 71.8 mm, 72 parts, among them J1 Power IN, J3 Power OUT, J4 OLED I2C, J5 PDI, J6 OLED, SW1 SW_DIP_x01, U1 INA169, U2 LMZ14203H, U3 L78M12, U4 INA169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

Commit message: Software init commit
Connections:
- J5 pad 1: PDI_CLK -> PDI_DATA
- J5 pad 5: PDI_DATA -> PDI_CLK
Routing:
- net PDI_DATA: track 45.4 -> 41.7 mm
- net GND: track 272.0 -> 275.4 mm
- net PDI_CLK: track 46.5 -> 44.0 mm
Other:
- board text added: "Vin"
- board text added: "Vout"
Changed lines of the file:
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@@
   (general
     (thickness 1.6)
-    (drawings 8)
-    (tracks 610)
+    (drawings 10)
+    (tracks 607)
     (zones 0)
     (modules 72)
@@
     (38 B.Mask user)
     (39 F.Mask user)
-    (40 Dwgs.User user)
-    (41 Cmts.User user)
-    (42 Eco1.User user)
-    (43 Eco2.User user)
+    (40 Dwgs.User user hide)
+    (41 Cmts.User user hide)
+    (42 Eco1.User user hide)
+    (43 Eco2.User user hide)
     (44 Edge.Cuts user)
-    (45 Margin user)
-    (46 B.CrtYd user)
-    (47 F.CrtYd user)
+    (45 Margin user hide)
+    (46 B.CrtYd user hide)
+    (47 F.CrtYd user hide)
     (48 B.Fab user)
-    (49 F.Fab user)
+    (49 F.Fab user hide)
   )
   (setup
@@
     (pad_to_mask_clearance 0.2)
     (aux_axis_origin 0 0)
-    (visible_elements 7FFFFF9F)
+    (visible_elements 7FFFFFBF)
     (pcbplotparams
-      (layerselection 0x01000_ffffffff)
+      (layerselection 0x010c0_ffffffff)
       (usegerberextensions false)
       (usegerberattributes false)
@@
       (net 14 GND))
     (pad 5 thru_hole oval (at 0 5.08 180) (size 2 2) (drill 1) (layers *.Cu *.Mask)
-      (net 23 PDI_DATA))
+      (net 24 PDI_CLK))
     (pad 4 thru_hole oval (at 2.54 2.54 180) (size 1 1) (drill 1) (layers *.Cu *.Mask))
     (pad 3 thru_hole oval (at 0 2.54 180) (size 1 1) (drill 1) (layers *.Cu *.Mask))
@@
       (net 18 +3V3))
     (pad 1 thru_hole rect (at 0 0 180) (size 2 2) (drill 1) (layers *.Cu *.Mask)
-      (net 24 PDI_CLK))
+      (net 23 PDI_DATA))
     (model ${KISYS3DMOD}/Pin_Headers.3dshapes/Pin_Header_Straight_2x03_Pitch2.54mm.wrl
       (at (xyz 0 0 0))
@@
       (clearance 3.25))
   )
+  (gr_text Vout (at 105.41 78.105) (layer F.Cu)
+    (effects (font (size 2.54 2.54) (thickness 0.508)))
+  )
+  (gr_text Vin (at 78.74 78.105) (layer F.Cu)
+    (effects (font (size 2.54 2.54) (thickness 0.508)))
+  )
   (gr_text JP (at 133.985 107.95) (layer B.Cu)
     (effects (font (size 2.032 2.032) (thickness 0.508)) (justify mirror))
@@
   (segment (start 82.82 90.075) (end 85.09 92.345) (width 0.8128) (layer B.Cu) (net 14))
   (segment (start 82.82 89.535) (end 82.82 90.075) (width 0.8128) (layer B.Cu) (net 14))
+  (segment (start 101.2028 106.045) (end 97.79 106.045) (width 0.8128) (layer F.Cu) (net 14))
   (segment (start 65.659 69.358) (end 67.607 69.358) (width 0.8128) (layer B.Cu) (net 15) (status 400000))
   (segment (start 67.607 69.358) (end 67.607 68.242) (width 0.8128) (layer B.Cu) (net 15))
@@
   (segment (start 80.645 99.695) (end 85.725 99.695) (width 0.5588) (layer B.Cu) (net 22))
   (segment (start 85.725 99.695) (end 86.43 98.99) (width 0.5588) (layer B.Cu) (net 22))
-  (segment (start 135.255 94.615) (end 135.255 96.52) (width 0.5588) (layer B.Cu) (net 23))
   (segment (start 94.075 93.54) (end 94.075 92.396318) (width 0.5588) (layer B.Cu) (net 23))
   (segment (start 94.075 92.396318) (end 94.396318 92.075) (width 0.5588) (layer B.Cu) (net 23))
@@
   (segment (start 113.665 92.075) (end 114.935 93.345) (width 0.5588) (layer B.Cu) (net 23))
   (segment (start 114.935 93.345) (end 133.985 93.345) (width 0.5588) (layer B.Cu) (net 23))
-  (segment (start 133.985 93.345) (end 135.255 94.615) (width 0.5588) (layer B.Cu) (net 23))
-  (segment (start 135.255 103.0088) (end 135.255 101.6) (width 0.5588) (layer B.Cu) (net 24))
   (segment (start 95.7088 93.54) (end 95.9038 93.345) (width 0.5588) (layer B.Cu) (net 24))
   (segment (start 94.875 93.54) (end 95.7088 93.54) (width 0.5588) (layer B.Cu) (net 24))
   (segment (start 95.9038 93.345) (end 112.395 93.345) (width 0.5588) (layer B.Cu) (net 24))
-  (segment (start 134.4438 103.82) (end 135.255 103.0088) (width 0.5588) (layer B.Cu) (net 24))
   (segment (start 122.87 103.82) (end 134.4438 103.82) (width 0.5588) (layer B.Cu) (net 24))
   (segment (start 112.395 93.345) (end 122.87 103.82) (width 0.5588) (layer B.Cu) (net 24))
