File: KiCad/Power Supply LMZ14203H/Power Supply LMZ14203H.kicad_pcb (KiCad board)
At the start: 2 copper layers, 92.7 x 71.8 mm, 72 parts, among them J1 Power IN, J3 Power OUT, J4 OLED I2C, J5 PDI, J6 OLED, SW1 SW_DIP_x01, U1 INA169, U2 LMZ14203H, U3 L78M12, U4 INA169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

Commit message: PCb fixes
Parts:
- C25, C27: value 100n -> 1u
- R1: value 90k -> 68k
- R15, R4: value 10k -> 20k
- R2: value 10k -> 2k2
Connections:
- C24 pad 1: Net-(C24-Pad1) -> +3V3
- J6 pad 19: Net-(C24-Pad1) -> +3V3
- J6 pad 20: Net-(C24-Pad1) -> +3V3
- J6 pad 21: Net-(C24-Pad1) -> +3V3
Routing:
- net Net-(C24-Pad1): track 9.11 -> 0.00 mm, vias 1 -> 0
- net +3V3: track 135.9 -> 145.0 mm, vias 4 -> 5
