File: KiCad/MobilePowerBank/MobilePowerBank.sch (KiCad schematic (older format))
At the start: 120 parts, among them J1 Power IN, J2 Power OUT, J3 Power OUT, J4 OLED I2C, J5 PDI, J6 OLED, J7 Power OUT, SW1 SW_DIP_x01, U1 INA169, U10 INA138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

Commit message: 5 power supplies created
Parts:
- added C45, C46: 100u, Capacitors_Tantalum_SMD:CP_Tantalum_Case-V_EIA-7343-20_Wave, symbol Device:CP
- added C47, C48: 10u/35V/X7R, Capacitors_SMD:C_2220, symbol Device:C
- added C49, C50: 4u7, Capacitors_SMD:C_0805, symbol Device:C
- added C51, C52: 22n, Capacitors_SMD:C_0805, symbol Device:C
- added C53, C54, C55, C56: 47u/1-45mESR, Capacitors_Tantalum_SMD:CP_Tantalum_Case-D_EIA-7343-31_Reflow, symbol Device:CP
- added C57, C58, C59, C60: 100n, Capacitors_SMD:C_0805, symbol Device:C
- added C61, C62: 1u, Capacitors_SMD:C_0805, symbol Device:C
- added J8: Power OUT 4, Connectors_Terminal_Blocks:TerminalBlock_Altech_AK300-2_P5.00mm, symbol conn:Conn_01x02
- added J9: Power OUT 5, Connectors_Terminal_Blocks:TerminalBlock_Altech_AK300-2_P5.00mm, symbol conn:Conn_01x02
- added R56, R58: 220k, Resistors_SMD:R_0805, symbol Device:R
- added R57, R59, R60, R62: 30k, Resistors_SMD:R_0805, symbol Device:R
- added R61, R63: 300k, Resistors_SMD:R_0805, symbol Device:R
- added R64, R65, R82, R83: 20k, Resistors_SMD:R_0805, symbol Device:R
- added R66, R67: 2k2, Resistors_SMD:R_0805, symbol Device:R
- added R68, R69, R70, R71: 15k4, Resistors_SMD:R_0805, symbol Device:R
- added R72, R74: 90k, Resistors_SMD:R_0805, symbol Device:R
- added R73, R75: 10k, Resistors_SMD:R_0805, symbol Device:R
- added R76, R77, R78, R79, R80, R81: 0R1, Resistors_SMD:R_2512, symbol Device:R
- added U11, U12: LMZ14201H, TO_SOT_Packages_SMD:TO-263-7_TabPin4, symbol myLib:LMZ14203H
- added U13, U14: INA138, TO_SOT_Packages_SMD:SOT-23-5, symbol myLib:INA169
- added U15: ATXMEGA256A3U-AU, Housings_QFP:TQFP-64_14x14mm_Pitch0.8mm, symbol atmel:ATXMEGA256A3U-AU
- J2: value Power OUT -> Power OUT 2
- J3: value Power OUT -> Power OUT 1
- J7: value Power OUT -> Power OUT 3
Connections:
- net labels added: OUT_1_Current, OUT_1_Voltage, OUT_2_Current, OUT_2_Voltage, OUT_3_Current, OUT_3_Voltage, OUT_4_Current, OUT_4_Voltage, OUT_5_Current, OUT_5_Voltage, POWER_4_OUT, POWER_5_OUT
- wire segments 383 -> 535
Other:
- note added: "Vout = 12V\nIout(max) = 1A"

Commit message: xmega added
Parts:
- removed U6: ATXMEGA32E5-AU, Housings_QFP:TQFP-32_7x7mm_Pitch0.8mm, symbol atmel:ATXMEGA32E5-AU
- added C63, C65, C67, C69: 100n, Capacitors_SMD:C_0805, symbol Device:C
- added C64, C66, C68, C70: 10u, Capacitors_Tantalum_SMD:CP_Tantalum_Case-B_EIA-3528-21_Wave, symbol Device:CP
- C1, C11, C28, C45, C46: value 100u -> 47u
- C13: value 100n -> 47u
- C14: footprint Capacitors_SMD:CP_Elec_6.3x7.7 -> Capacitors_Tantalum_SMD:CP_Tantalum_Case-V_EIA-7343-20_Wave
- C17: footprint Capacitors_SMD:CP_Elec_6.3x5.8 -> Capacitors_Tantalum_SMD:CP_Tantalum_Case-V_EIA-7343-20_Wave
- C19, C21, C22, C23: footprint Capacitors_SMD:CP_Elec_4x5.8 -> Capacitors_Tantalum_SMD:CP_Tantalum_Case-B_EIA-3528-21_Wave
- C5: value 100u -> 47u; footprint Capacitors_SMD:CP_Elec_6.3x7.7 -> Capacitors_Tantalum_SMD:CP_Tantalum_Case-V_EIA-7343-20_Wave
- SW1: footprint Buttons_Switches_SMD:SW_SPST_B3S-1000 -> Pin_Headers:Pin_Header_Angled_1x02_Pitch2.54mm
Connections:
- net labels added: VDD
- wire segments 535 -> 560
- no-connect marks 16 -> 11
Other:
- moved on the sheet: U15

Commit message: PCB major work
Parts:
- added C71: 47u, Capacitors_Tantalum_SMD:CP_Tantalum_Case-V_EIA-7343-20_Wave, symbol Device:CP
- added C72: 10u/35V/X7R, Capacitors_SMD:C_2220, symbol Device:C
- added C73: 4u7, Capacitors_SMD:C_0805, symbol Device:C
- added C74: 22n, Capacitors_SMD:C_0805, symbol Device:C
- added C75, C76: 47u/1-45mESR, Capacitors_Tantalum_SMD:CP_Tantalum_Case-D_EIA-7343-31_Reflow, symbol Device:CP
- added C77, C78: 100n, Capacitors_SMD:C_0805, symbol Device:C
- added C79: 1u, Capacitors_SMD:C_0805, symbol Device:C
- added J10: Power OUT 6, Connectors_Terminal_Blocks:TerminalBlock_Altech_AK300-2_P5.00mm, symbol conn:Conn_01x02
- added R84: 220k, Resistors_SMD:R_0805, symbol Device:R
- added R85, R86: 30k, Resistors_SMD:R_0805, symbol Device:R
- added R87: 300k, Resistors_SMD:R_0805, symbol Device:R
- added R88, R97: 20k, Resistors_SMD:R_0805, symbol Device:R
- added R89: 2k2, Resistors_SMD:R_0805, symbol Device:R
- added R90, R91: 15k4, Resistors_SMD:R_0805, symbol Device:R
- added R92: 90k, Resistors_SMD:R_0805, symbol Device:R
- added R93: 10k, Resistors_SMD:R_0805, symbol Device:R
- added R94, R95, R96: 0R1, Resistors_SMD:R_2512, symbol Device:R
- added R98: 0, Resistors_SMD:R_0805, symbol Device:R
- added U16: INA138, TO_SOT_Packages_SMD:SOT-23-5, symbol myLib:INA169
- added U6: LMZ14203H, TO_SOT_Packages_SMD:TO-263-7_TabPin4, symbol myLib:LMZ14203H
- added x1, x2, x3, x4: jumper, JPJumpers:Jumper_30x1.5, symbol myJumpers:jumper
- added x5: jumper, JPJumpers:Jumper_45x1.5, symbol myJumpers:jumper
Connections:
- net labels added: OUT_6_Current, OUT_6_Voltage, POWER_6_OUT, POWER_IN_1, POWER_IN_3, POWER_IN_4, POWER_IN_6
- wire segments 560 -> 658
Other:
- moved on the sheet: U15

Commit message: PCB finish, BOM check
Parts:
- added x6, x7, x8, x9: jumper, JPJumpers:Jumper_30x1.5, symbol myJumpers:jumper
- C1, C11, C28, C45, C46, C5, C71: value 47u -> 47u/35V
- C13: value 47u -> 100n
- C14: value 100u -> 47u/16V
- C17: value 47u -> 47u/6.3V
- C19, C21, C64, C66, C68, C70: value 10u -> 10u/6.3V
- C22, C23: value 10u -> 10u/16V
- R14, R16, R17, R18, R19, R3, R48, R49, R50, R51, R52, R53, R76, R77, R78, R79, R80, R81, R94, R95, R96: value 0R1 -> 0R033
Connections:
- net labels removed: OUT_Current, OUT_Voltage
- wire segments 658 -> 654

Commit message: Cap changed
Parts:
- R22: value 15k4 -> 47k
- R27: value 220k -> 300k
- R28: value 15k4 -> 4k7
- R29, R31, R57, R59, R85: value 30k -> 47k
- R5: value 30k -> 100k
- R6: value 30k -> 68k
- U1: value INA169 -> INA139
- U10, U13, U14, U16, U4, U9: value INA138 -> INA139
Other:
- note added: "Vout = 19.6V\nIout(max) = 3A\nUen = 22.9V"

Commit message: Aligning PCB
Parts:
- removed C75, C76: 47u/1-45mESR, Capacitors_Tantalum_SMD:CP_Tantalum_Case-D_EIA-7343-31_Reflow, symbol Device:CP
- added C80: 1u/50V, Capacitors_SMD:C_0805, symbol Device:C
- added C81: 100u/6V3, Capacitors_SMD:C_1812, symbol Device:C
- added MH1, MH2, MH3, MH4: MountingHole_Pad, Mounting_Holes:MountingHole_3.5mm, symbol Mechanical:MountingHole_Pad
- C14, C17: footprint Capacitors_Tantalum_SMD:CP_Tantalum_Case-V_EIA-7343-20_Wave -> Capacitors_Tantalum_SMD:CP_Tantalum_Case-C_EIA-6032-28_Wave
- C2, C29, C30, C47, C48, C72: value 10u/35V/X7R -> 10u/50V/X7R
- C3: value 4u7 -> 4n7
- C31, C32: value 4u7 -> 10n
- C73: value 4u7 -> 22n
- R84: value 220k -> 0
- R85: value 47k -> 0
- R86: value 30k -> 100k
- R87: value 300k -> 68k
- R88: value 20k -> 11k
- R89: value 2k2 -> 1k5
- R90: value 15k4 -> 7k68
- R91: value 15k4 -> 200
- U6: value LMZ14203H -> LMZ14203
Other:
- note added: "ASI1600\nVout = 12V\nIout(max) = 3A\nSS 2"
- note added: "Dell\nVout = 19.6V\nIout(max) = 3A\nUen = 22.9V\nSS 1 (Soft start order)"
- note added: "EQ6-R\nVout = 12V\nIout(max) = 3A\nSS 2"
- note added: "FlatField\nVout = 12V\nIout(max) = 1A\nSS 1"
- note added: "Moonlite\nVout = 12V\nIout(max) = 1A\nSS 1"
- note added: "USB\nVout = 5V\nIout(max) = 3A\nss 3"
- note removed: "Vout = 12V\nIout(max) = 1A"
- note removed: "Vout = 12V\nIout(max) = 3A"
- note removed: "Vout = 19.6V\nIout(max) = 3A\nUen = 22.9V"

Commit message: Pimping PCB
Parts:
- C1, C11, C28, C45, C46, C5, C71: footprint Capacitors_Tantalum_SMD:CP_Tantalum_Case-V_EIA-7343-20_Wave -> Capacitors_Tantalum_SMD:CP_Tantalum_Case-D_EIA-7343-31_Reflow
- C14, C17: footprint Capacitors_Tantalum_SMD:CP_Tantalum_Case-C_EIA-6032-28_Wave -> Capacitors_Tantalum_SMD:CP_Tantalum_Case-C_EIA-6032-28_Reflow
- C19, C21, C22, C23, C64, C66, C68, C70: footprint Capacitors_Tantalum_SMD:CP_Tantalum_Case-B_EIA-3528-21_Wave -> Capacitors_Tantalum_SMD:CP_Tantalum_Case-B_EIA-3528-21_Reflow
- C80: footprint Capacitors_SMD:C_0805 -> Capacitors_SMD:C_1206
- x1, x2, x3, x4, x6, x7, x8: footprint JPJumpers:Jumper_30x1.5 -> JPJumpers:Jumper_33x1.5
- x9: footprint JPJumpers:Jumper_30x1.5 -> JPJumpers:Jumper_45x1.5
Changed lines of the file:
@@
 F 0 "C1" H 5075 2650 50  0000 L CNN
 F 1 "47u/35V" H 5075 2450 50  0000 L CNN
-F 2 "Capacitors_Tantalum_SMD:CP_Tantalum_Case-V_EIA-7343-20_Wave" H 5088 2400 50  0001 C CNN
+F 2 "Capacitors_Tantalum_SMD:CP_Tantalum_Case-D_EIA-7343-31_Reflow" H 5088 2400 50  0001 C CNN
 F 3 "" H 5050 2550 50  0001 C CNN
 	1    5050 2550
@@
 F 0 "C19" H 12175 11350 50  0000 L CNN
 F 1 "10u/6.3V" H 12175 11150 50  0000 L CNN
-F 2 "Capacitors_Tantalum_SMD:CP_Tantalum_Case-B_EIA-3528-21_Wave" H 12188 11100 50  0001 C CNN
+F 2 "Capacitors_Tantalum_SMD:CP_Tantalum_Case-B_EIA-3528-21_Reflow" H 12188 11100 50  0001 C CNN
 F 3 "" H 12150 11250 50  0001 C CNN
 	1    12150 11250
@@
 F 0 "C21" H 13175 11350 50  0000 L CNN
 F 1 "10u/6.3V" H 13175 11150 50  0000 L CNN
-F 2 "Capacitors_Tantalum_SMD:CP_Tantalum_Case-B_EIA-3528-21_Wave" H 13188 11100 50  0001 C CNN
+F 2 "Capacitors_Tantalum_SMD:CP_Tantalum_Case-B_EIA-3528-21_Reflow" H 13188 11100 50  0001 C CNN
 F 3 "" H 13150 11250 50  0001 C CNN
 	1    13150 11250
@@
 F 0 "C14" H 3775 11700 50  0000 L CNN
 F 1 "47u/16V" H 3775 11500 50  0000 L CNN
-F 2 "Capacitors_Tantalum_SMD:CP_Tantalum_Case-C_EIA-6032-28_Wave" H 3788 11450 50  0001 C CNN
+F 2 "Capacitors_Tantalum_SMD:CP_Tantalum_Case-C_EIA-6032-28_Reflow" H 3788 11450 50  0001 C CNN
 F 3 "" H 3750 11600 50  0001 C CNN
 	1    3750 11600
@@
 F 0 "C17" H 5125 11700 50  0000 L CNN
 F 1 "47u/6.3V" H 5125 11500 50  0000 L CNN
-F 2 "Capacitors_Tantalum_SMD:CP_Tantalum_Case-C_EIA-6032-28_Wave" H 5138 11450 50  0001 C CNN
+F 2 "Capacitors_Tantalum_SMD:CP_Tantalum_Case-C_EIA-6032-28_Reflow" H 5138 11450 50  0001 C CNN
 F 3 "" H 5100 11600 50  0001 C CNN
 	1    5100 11600
@@
 F 0 "C5" H 2475 11700 50  0000 L CNN
 F 1 "47u/35V" H 2475 11500 50  0000 L CNN
-F 2 "Capacitors_Tantalum_SMD:CP_Tantalum_Case-V_EIA-7343-20_Wave" H 2488 11450 50  0001 C CNN
+F 2 "Capacitors_Tantalum_SMD:CP_Tantalum_Case-D_EIA-7343-31_Reflow" H 2488 11450 50  0001 C CNN
 F 3 "" H 2450 11600 50  0001 C CNN
 	1    2450 11600
@@
 F 0 "C23" H 16375 12450 50  0000 L CNN
 F 1 "10u/16V" H 16375 12250 50  0000 L CNN
-F 2 "Capacitors_Tantalum_SMD:CP_Tantalum_Case-B_EIA-3528-21_Wave" H 16388 12200 50  0001 C CNN
+F 2 "Capacitors_Tantalum_SMD:CP_Tantalum_Case-B_EIA-3528-21_Reflow" H 16388 12200 50  0001 C CNN
 F 3 "" H 16350 12350 50  0001 C CNN
 	1    16350 12350
@@
 F 0 "C22" H 16075 12450 50  0000 L CNN
 F 1 "10u/16V" H 16075 12250 50  0000 L CNN
-F 2 "Capacitors_Tantalum_SMD:CP_Tantalum_Case-B_EIA-3528-21_Wave" H 16088 12200 50  0001 C CNN
+F 2 "Capacitors_Tantalum_SMD:CP_Tantalum_Case-B_EIA-3528-21_Reflow" H 16088 12200 50  0001 C CNN
 F 3 "" H 16050 12350 50  0001 C CNN
 	1    16050 12350
@@
 F 0 "C11" H 5075 5250 50  0000 L CNN
 F 1 "47u/35V" H 5075 5050 50  0000 L CNN
-F 2 "Capacitors_Tantalum_SMD:CP_Tantalum_Case-V_EIA-7343-20_Wave" H 5088 5000 50  0001 C CNN
+F 2 "Capacitors_Tantalum_SMD:CP_Tantalum_Case-D_EIA-7343-31_Reflow" H 5088 5000 50  0001 C CNN
 F 3 "" H 5050 5150 50  0001 C CNN
 	1    5050 5150
@@
 F 0 "C28" H 5075 7700 50  0000 L CNN
 F 1 "47u/35V" H 5075 7500 50  0000 L CNN
-F 2 "Capacitors_Tantalum_SMD:CP_Tantalum_Case-V_EIA-7343-20_Wave" H 5088 7450 50  0001 C CNN
+F 2 "Capacitors_Tantalum_SMD:CP_Tantalum_Case-D_EIA-7343-31_Reflow" H 5088 7450 50  0001 C CNN
 F 3 "" H 5050 7600 50  0001 C CNN
 	1    5050 7600
@@
 F 0 "C45" H 11975 2700 50  0000 L CNN
 F 1 "47u/35V" H 11975 2500 50  0000 L CNN
-F 2 "Capacitors_Tantalum_SMD:CP_Tantalum_Case-V_EIA-7343-20_Wave" H 11988 2450 50  0001 C CNN
+F 2 "Capacitors_Tantalum_SMD:CP_Tantalum_Case-D_EIA-7343-31_Reflow" H 11988 2450 50  0001 C CNN
 F 3 "" H 11950 2600 50  0001 C CNN
 	1    11950 2600
@@
 F 0 "C46" H 11975 5250 50  0000 L CNN
 F 1 "47u/35V" H 11975 5050 50  0000 L CNN
-F 2 "Capacitors_Tantalum_SMD:CP_Tantalum_Case-V_EIA-7343-20_Wave" H 11988 5000 50  0001 C CNN
+F 2 "Capacitors_Tantalum_SMD:CP_Tantalum_Case-D_EIA-7343-31_Reflow" H 11988 5000 50  0001 C CNN
 F 3 "" H 11950 5150 50  0001 C CNN
 	1    11950 5150
@@
 F 0 "C70" H 12175 10850 50  0000 L CNN
 F 1 "10u/6.3V" H 12175 10650 50  0000 L CNN
-F 2 "Capacitors_Tantalum_SMD:CP_Tantalum_Case-B_EIA-3528-21_Wave" H 12188 10600 50  0001 C CNN
+F 2 "Capacitors_Tantalum_SMD:CP_Tantalum_Case-B_EIA-3528-21_Reflow" H 12188 10600 50  0001 C CNN
 F 3 "" H 12150 10750 50  0001 C CNN
 	1    12150 10750
@@
 F 0 "C68" H 12175 10350 50  0000 L CNN
 F 1 "10u/6.3V" H 12175 10150 50  0000 L CNN
-F 2 "Capacitors_Tantalum_SMD:CP_Tantalum_Case-B_EIA-3528-21_Wave" H 12188 10100 50  0001 C CNN
+F 2 "Capacitors_Tantalum_SMD:CP_Tantalum_Case-B_EIA-3528-21_Reflow" H 12188 10100 50  0001 C CNN
 F 3 "" H 12150 10250 50  0001 C CNN
 	1    12150 10250
@@
 F 0 "C66" H 12175 9850 50  0000 L CNN
 F 1 "10u/6.3V" H 12175 9650 50  0000 L CNN
-F 2 "Capacitors_Tantalum_SMD:CP_Tantalum_Case-B_EIA-3528-21_Wave" H 12188 9600 50  0001 C CNN
+F 2 "Capacitors_Tantalum_SMD:CP_Tantalum_Case-B_EIA-3528-21_Reflow" H 12188 9600 50  0001 C CNN
 F 3 "" H 12150 9750 50  0001 C CNN
 	1    12150 9750
@@
 F 0 "C64" H 12175 9350 50  0000 L CNN
 F 1 "10u/6.3V" H 12175 9150 50  0000 L CNN
-F 2 "Capacitors_Tantalum_SMD:CP_Tantalum_Case-B_EIA-3528-21_Wave" H 12188 9100 50  0001 C CNN
+F 2 "Capacitors_Tantalum_SMD:CP_Tantalum_Case-B_EIA-3528-21_Reflow" H 12188 9100 50  0001 C CNN
 F 3 "" H 12150 9250 50  0001 C CNN
 	1    12150 9250
@@
 F 0 "C71" H 13875 8100 50  0000 L CNN
 F 1 "47u/35V" H 13875 7900 50  0000 L CNN
-F 2 "Capacitors_Tantalum_SMD:CP_Tantalum_Case-V_EIA-7343-20_Wave" H 13888 7850 50  0001 C CNN
+F 2 "Capacitors_Tantalum_SMD:CP_Tantalum_Case-D_EIA-7343-31_Reflow" H 13888 7850 50  0001 C CNN
 F 3 "" H 13850 8000 50  0001 C CNN
 	1    13850 8000
@@
 F 0 "x1" H 4900 7325 50  0000 C CNN
 F 1 "jumper" H 4900 7234 50  0000 C CNN
-F 2 "JPJumpers:Jumper_30x1.5" H 4900 7200 50  0001 C CNN
+F 2 "JPJumpers:Jumper_33x1.5" H 4900 7200 50  0001 C CNN
 F 3 "" H 4900 7200 50  0001 C CNN
 	1    4900 7200
@@
 F 0 "x2" H 4900 2275 50  0000 C CNN
 F 1 "jumper" H 4900 2184 50  0000 C CNN
-F 2 "JPJumpers:Jumper_30x1.5" H 4900 2150 50  0001 C CNN
+F 2 "JPJumpers:Jumper_33x1.5" H 4900 2150 50  0001 C CNN
 F 3 "" H 4900 2150 50  0001 C CNN
 	1    4900 2150
@@
 F 0 "x3" H 11800 2325 50  0000 C CNN
 F 1 "jumper" H 11800 2234 50  0000 C CNN
-F 2 "JPJumpers:Jumper_30x1.5" H 11800 2200 50  0001 C CNN
+F 2 "JPJumpers:Jumper_33x1.5" H 11800 2200 50  0001 C CNN
 F 3 "" H 11800 2200 50  0001 C CNN
 	1    11800 2200
@@
 F 0 "x4" H 13700 7725 50  0000 C CNN
 F 1 "jumper" H 13700 7634 50  0000 C CNN
-F 2 "JPJumpers:Jumper_30x1.5" H 13700 7600 50  0001 C CNN
+F 2 "JPJumpers:Jumper_33x1.5" H 13700 7600 50  0001 C CNN
 F 3 "" H 13700 7600 50  0001 C CNN
 	1    13700 7600
@@
 F 0 "x7" H 19550 2825 50  0000 C CNN
 F 1 "jumper" H 19550 2734 50  0000 C CNN
-F 2 "JPJumpers:Jumper_30x1.5" H 19550 2700 50  0001 C CNN
+F 2 "JPJumpers:Jumper_33x1.5" H 19550 2700 50  0001 C CNN
 F 3 "" H 19550 2700 50  0001 C CNN
 	1    19550 2700
@@
 F 0 "x6" H 19550 2575 50  0000 C CNN
 F 1 "jumper" H 19550 2484 50  0000 C CNN
-F 2 "JPJumpers:Jumper_30x1.5" H 19550 2450 50  0001 C CNN
+F 2 "JPJumpers:Jumper_33x1.5" H 19550 2450 50  0001 C CNN
 F 3 "" H 19550 2450 50  0001 C CNN
 	1    19550 2450
@@
 F 0 "x9" H 19550 2375 50  0000 C CNN
 F 1 "jumper" H 19550 2284 50  0000 C CNN
-F 2 "JPJumpers:Jumper_30x1.5" H 19550 2250 50  0001 C CNN
+F 2 "JPJumpers:Jumper_45x1.5" H 19550 2250 50  0001 C CNN
 F 3 "" H 19550 2250 50  0001 C CNN
 	1    19550 2250
@@
 F 0 "x8" H 19550 2125 50  0000 C CNN
 F 1 "jumper" H 19550 2034 50  0000 C CNN
-F 2 "JPJumpers:Jumper_30x1.5" H 19550 2000 50  0001 C CNN
+F 2 "JPJumpers:Jumper_33x1.5" H 19550 2000 50  0001 C CNN
 F 3 "" H 19550 2000 50  0001 C CNN
 	1    19550 2000
@@
 F 0 "C80" H 16475 8100 50  0000 L CNN
 F 1 "1u/50V" H 16475 7900 50  0000 L CNN
-F 2 "Capacitors_SMD:C_0805" H 16488 7850 50  0001 C CNN
+F 2 "Capacitors_SMD:C_1206" H 16488 7850 50  0001 C CNN
 F 3 "" H 16450 8000 50  0001 C CNN
 	1    16450 8000
@@
 	1    0    0    -1
 $EndComp
-Wire Bus Line
-	14300 13950 14300 15650
-Wire Bus Line
-	10800 13650 10800 15650
-Wire Bus Line
-	16800 12300 16800 13950
 $Comp
 L Mechanical:MountingHole_Pad MH1
@@
 	1    0    0    -1
 $EndComp
+Wire Bus Line
+	14300 13950 14300 15650
+Wire Bus Line
+	10800 13650 10800 15650
+Wire Bus Line
+	16800 12300 16800 13950
 $EndSCHEMATC

Commit message: Pimping PCB
Parts:
- added C75: 330n / 50V, Capacitors_SMD:C_0805, symbol Device:C
- added C76: 47u/16V, Capacitors_SMD:CP_Elec_4x5.8, symbol Device:CP
- added C82, C83, C84, C85, C86: 1u/50V, Capacitors_SMD:C_1206, symbol Device:C
- added J11: PowerLED, Connectors_JST:JST_XH_B02B-XH-A_02x2.50mm_Straight, symbol conn:Conn_01x02
- added R99: 1k, Resistors_SMD:R_0805, symbol Device:R
- added U17: L78L05_SOT89, TO_SOT_Packages_SMD:SOT-89-3, symbol regul:L78L05_SOT89
Connections:
- net labels added: Unfused_Power
- wire segments 654 -> 703
Other:
- note added: "R=5V/5mA=1k"
