File: KiCad/MobilePowerBank/MobilePowerBank.sch (KiCad schematic (older format))
At the start: 230 parts, among them J1 Power IN, J10 Power OUT 6, J11 PowerLED, J2 Power OUT 2, J3 Power OUT 1, J4 OLED I2C, J5 PDI, J6 OLED, J7 Power OUT 3, J8 Power OUT 4, J9 Power OUT 5, SW1 SW_DIP_x01, U1 INA139, U10 INA139, U11 LMZ14201H, U12 LMZ14201H, U13 INA139, U14 INA139, U15 ATXMEGA256A3U-AU, U16 INA139, U17 L78L05_SOT89, U2 LMZ14203H, U3 L78M12, U4 INA139, U5 UA78M33, U6 LMZ14203, U7 LMZ14203H, U8 LMZ14203H, U9 INA139, x1 jumper, x2 jumper, x3 jumper, x4 jumper, x5 jumper, x6 jumper, x7 jumper, x8 jumper, x9 jumper

Commit message: DMA and screen
Parts:
- R44: value 90k -> 47k
- R45: value 10k -> 3k9
Other:
- note added: "3.9/(47+3.9) * 12V = 0.92V"
Changed lines of the file:
@@
 P 7950 4000
 F 0 "R44" V 8030 4000 50  0000 C CNN
-F 1 "90k" V 7950 4000 50  0000 C CNN
+F 1 "47k" V 7950 4000 50  0000 C CNN
 F 2 "Resistors_SMD:R_0805" V 7880 4000 50  0001 C CNN
 F 3 "" H 7950 4000 50  0001 C CNN
@@
 P 7950 4400
 F 0 "R45" V 8030 4400 50  0000 C CNN
-F 1 "10k" V 7950 4400 50  0000 C CNN
+F 1 "3k9" V 7950 4400 50  0000 C CNN
 F 2 "Resistors_SMD:R_0805" V 7880 4400 50  0001 C CNN
 F 3 "" H 7950 4400 50  0001 C CNN
@@
 Wire Bus Line
 	16800 12300 16800 13950
+Text Notes 6750 4500 0    50   ~ 0
+3.9/(47+3.9) * 12V = 0.92V
 $EndSCHEMATC

Commit message: Support for Output 3 added
Parts:
- C76: value 47u/16V -> 22u/16V
- J1, J10, J11, J2, J3, J7, J8, J9: symbol conn:Conn_01x02 -> MobilePowerBank-rescue:Conn_01x02-conn
- J4: symbol conn:Conn_01x04 -> MobilePowerBank-rescue:Conn_01x04-conn
- J5: symbol conn:Conn_02x03_Odd_Even -> MobilePowerBank-rescue:Conn_02x03_Odd_Even-conn
- J6: symbol conn:Conn_01x30 -> MobilePowerBank-rescue:Conn_01x30-conn
- R99: value 1k -> 3k3
- SW1: symbol switches:SW_DIP_x01 -> MobilePowerBank-rescue:SW_DIP_x01-switches
- U15: symbol atmel:ATXMEGA256A3U-AU -> MobilePowerBank-rescue:ATXMEGA256A3U-AU-atmel
- U17: symbol regul:L78L05_SOT89 -> MobilePowerBank-rescue:L78L05_SOT89-regul
- U3, U5: symbol regul:L7805 -> MobilePowerBank-rescue:L7805-regul
- x1, x2, x3, x4, x5, x6, x7, x8, x9: symbol myJumpers:jumper -> MobilePowerBank-rescue:jumper-myJumpers
Changed lines of the file:
@@
 $EndComp
 $Comp
-L conn:Conn_01x02 J1
+L MobilePowerBank-rescue:Conn_01x02-conn J1
 U 1 1 59FFC4D5
 P 850 5400
@@
 $EndComp
 $Comp
-L conn:Conn_01x02 J3
+L MobilePowerBank-rescue:Conn_01x02-conn J3
 U 1 1 59FFC5CF
 P 9400 2450
@@
 Connection ~ 11450 11850
 $Comp
-L conn:Conn_02x03_Odd_Even J5
+L MobilePowerBank-rescue:Conn_02x03_Odd_Even-conn J5
 U 1 1 5B7326AC
 P 6700 11550
@@
 NoConn ~ 6500 11550
 $Comp
-L conn:Conn_01x04 J4
+L MobilePowerBank-rescue:Conn_01x04-conn J4
 U 1 1 5B733C01
 P 6400 12600
@@
 	13750 13650 13550 13650
 $Comp
-L regul:L7805 U3
+L MobilePowerBank-rescue:L7805-regul U3
 U 1 1 5B736775
 P 3100 11350
@@
 $EndComp
 $Comp
-L regul:L7805 U5
+L MobilePowerBank-rescue:L7805-regul U5
 U 1 1 5B73681E
 P 4450 11350
@@
 $EndComp
 $Comp
-L switches:SW_DIP_x01 SW1
+L MobilePowerBank-rescue:SW_DIP_x01-switches SW1
 U 1 1 5B739FEE
 P 4100 13000
@@
 Connection ~ 4100 12600
 $Comp
-L conn:Conn_01x30 J6
+L MobilePowerBank-rescue:Conn_01x30-conn J6
 U 1 1 5B73B056
 P 17750 13200
@@
 $EndComp
 $Comp
-L conn:Conn_01x02 J2
+L MobilePowerBank-rescue:Conn_01x02-conn J2
 U 1 1 5BEE7E91
 P 9400 5000
@@
 $EndComp
 $Comp
-L conn:Conn_01x02 J7
+L MobilePowerBank-rescue:Conn_01x02-conn J7
 U 1 1 5BF01E64
 P 9400 7500
@@
 $EndComp
 $Comp
-L conn:Conn_01x02 J8
+L MobilePowerBank-rescue:Conn_01x02-conn J8
 U 1 1 5BF3E2D5
 P 16300 2500
@@
 $EndComp
 $Comp
-L conn:Conn_01x02 J9
+L MobilePowerBank-rescue:Conn_01x02-conn J9
 U 1 1 5BF3E431
 P 16300 5050
@@
 $EndComp
 $Comp
-L atmel:ATXMEGA256A3U-AU U15
+L MobilePowerBank-rescue:ATXMEGA256A3U-AU-atmel U15
 U 1 1 5BF96E39
 P 12550 13250
@@
 $EndComp
 $Comp
-L conn:Conn_01x02 J10
+L MobilePowerBank-rescue:Conn_01x02-conn J10
 U 1 1 5BCA8471
 P 18200 7900
@@
 Connection ~ 8700 6300
 $Comp
-L myJumpers:jumper x1
+L MobilePowerBank-rescue:jumper-myJumpers x1
 U 1 1 5BFC2A6F
 P 4900 7200
@@
 Connection ~ 8700 3800
 $Comp
-L myJumpers:jumper x2
+L MobilePowerBank-rescue:jumper-myJumpers x2
 U 1 1 5C08F1E5
 P 4900 2150
@@
 POWER_IN_1
 $Comp
-L myJumpers:jumper x3
+L MobilePowerBank-rescue:jumper-myJumpers x3
 U 1 1 5C1BCF0A
 P 11800 2200
@@
 POWER_IN_4
 $Comp
-L myJumpers:jumper x4
+L MobilePowerBank-rescue:jumper-myJumpers x4
 U 1 1 5C80460D
 P 13700 7600
@@
 POWER_IN_6
 $Comp
-L myJumpers:jumper x5
+L MobilePowerBank-rescue:jumper-myJumpers x5
 U 1 1 5CA0F569
 P 2350 11250
@@
 $EndComp
 $Comp
-L myJumpers:jumper x7
+L MobilePowerBank-rescue:jumper-myJumpers x7
 U 1 1 5CA8A130
 P 19550 2700
@@
 $EndComp
 $Comp
-L myJumpers:jumper x6
+L MobilePowerBank-rescue:jumper-myJumpers x6
 U 1 1 5CA8B5EF
 P 19550 2450
@@
 $EndComp
 $Comp
-L myJumpers:jumper x9
+L MobilePowerBank-rescue:jumper-myJumpers x9
 U 1 1 5CAF3D77
 P 19550 2250
@@
 $EndComp
 $Comp
-L myJumpers:jumper x8
+L MobilePowerBank-rescue:jumper-myJumpers x8
 U 1 1 5CAF3D89
 P 19550 2000
@@
 $EndComp
 $Comp
-L regul:L78L05_SOT89 U17
+L MobilePowerBank-rescue:L78L05_SOT89-regul U17
 U 1 1 5C1B834B
 P 2150 6300
@@
 P 2700 6300
 F 0 "R99" V 2780 6300 50  0000 C CNN
-F 1 "1k" V 2700 6300 50  0000 C CNN
+F 1 "3k3" V 2700 6300 50  0000 C CNN
 F 2 "Resistors_SMD:R_0805" V 2630 6300 50  0001 C CNN
 F 3 "" H 2700 6300 50  0001 C CNN
@@
 P 3150 6500
 F 0 "C76" H 3175 6600 50  0000 L CNN
-F 1 "47u/16V" H 3175 6400 50  0000 L CNN
+F 1 "22u/16V" H 3175 6400 50  0000 L CNN
 F 2 "Capacitors_SMD:CP_Elec_4x5.8" H 3188 6350 50  0001 C CNN
 F 3 "" H 3150 6500 50  0001 C CNN
@@
 R=5V/5mA=1k
 $Comp
-L conn:Conn_01x02 J11
+L MobilePowerBank-rescue:Conn_01x02-conn J11
 U 1 1 5C8573AF
 P 3800 6300
@@
 Wire Wire Line
 	15100 5600 14850 5600
+Text Notes 6750 4500 0    50   ~ 0
+3.9/(47+3.9) * 12V = 0.92V
 Wire Bus Line
 	14300 13950 14300 15650
@@
 Wire Bus Line
 	16800 12300 16800 13950
-Text Notes 6750 4500 0    50   ~ 0
-3.9/(47+3.9) * 12V = 0.92V
 $EndSCHEMATC

Commit message: Five outputs callibration
Parts:
- R12: value 90k -> 100k
- R13: value 10k -> 4k7
Other:
- note added: "4.7/(100+4.7) * 12V = 0.90V"
Changed lines of the file:
@@
 P 8000 1450
 F 0 "R12" V 8080 1450 50  0000 C CNN
-F 1 "90k" V 8000 1450 50  0000 C CNN
+F 1 "100k" V 8000 1450 50  0000 C CNN
 F 2 "Resistors_SMD:R_0805" V 7930 1450 50  0001 C CNN
 F 3 "" H 8000 1450 50  0001 C CNN
@@
 P 8000 1850
 F 0 "R13" V 8080 1850 50  0000 C CNN
-F 1 "10k" V 8000 1850 50  0000 C CNN
+F 1 "4k7" V 8000 1850 50  0000 C CNN
 F 2 "Resistors_SMD:R_0805" V 7930 1850 50  0001 C CNN
 F 3 "" H 8000 1850 50  0001 C CNN
@@
 Wire Bus Line
 	16800 12300 16800 13950
+Text Notes 7050 1250 0    50   ~ 0
+4.7/(100+4.7) * 12V = 0.90V
 $EndSCHEMATC

Commit message: Storing data in EEPROM on power loss
Other:
- note added: "2k2/(2k2+68k)=0.03 (1/32)"
Changed lines of the file:
@@
 Text Notes 6750 4500 0    50   ~ 0
 3.9/(47+3.9) * 12V = 0.92V
+Text Notes 7050 1250 0    50   ~ 0
+4.7/(100+4.7) * 12V = 0.90V
 Wire Bus Line
 	14300 13950 14300 15650
@@
 Wire Bus Line
 	16800 12300 16800 13950
-Text Notes 7050 1250 0    50   ~ 0
-4.7/(100+4.7) * 12V = 0.90V
+Text Notes 950  4150 0    50   ~ 0
+2k2/(2k2+68k)=0.03  (1/32)
 $EndSCHEMATC

Commit message: Serial port added
Connections:
- net labels added: BT_A, BT_B, BT_RXD, BT_TXD
- wire segments 703 -> 707
Changed lines of the file:
@@
 	16800 13000 16900 12900
 Wire Bus Line
-	16800 13950 14300 13950
+	16800 14500 14300 14500
 Text Label 11450 14150 2    60   ~ 0
 OLED_D6
@@
 Text Notes 7050 1250 0    50   ~ 0
 4.7/(100+4.7) * 12V = 0.90V
+Text Notes 950  4150 0    50   ~ 0
+2k2/(2k2+68k)=0.03  (1/32)
+Text GLabel 13800 14150 2    50   Input ~ 0
+BT_RXD
+Text GLabel 13800 14250 2    50   Input ~ 0
+BT_TXD
+Wire Wire Line
+	13800 14150 13550 14150
+Wire Wire Line
+	13550 14250 13800 14250
+Text GLabel 13800 13750 2    50   Input ~ 0
+BT_A
+Text GLabel 13800 13950 2    50   Input ~ 0
+BT_B
+Wire Wire Line
+	13800 13750 13550 13750
+Wire Wire Line
+	13550 13950 13800 13950
 Wire Bus Line
-	14300 13950 14300 15650
+	14300 14500 14300 15650
 Wire Bus Line
 	10800 13650 10800 15650
 Wire Bus Line
-	16800 12300 16800 13950
-Text Notes 950  4150 0    50   ~ 0
-2k2/(2k2+68k)=0.03  (1/32)
+	16800 12300 16800 14500
 $EndSCHEMATC
