File: KiCad/MobilePowerBank/MobilePowerBank.kicad_pcb (KiCad board)
At the start: 2 copper layers, 136 x 211 mm, 220 parts, among them J1 Power IN, J10 Power OUT 6, J2 Power OUT 2, J3 Power OUT 1, J4 OLED I2C, J5 PDI, J6 OLED, J7 Power OUT 3, J8 Power OUT 4, J9 Power OUT 5, SW1 SW_DIP_x01, U1 INA139, U10 INA139, U11 LMZ14201H, U12 LMZ14201H, U13 INA139, U14 INA139, U15 ATXMEGA256A3U-AU, U16 INA139, U2 LMZ14203H, U3 L78M12, U4 INA139, U5 UA78M33, U6 LMZ14203, U7 LMZ14203H, U8 LMZ14203H, U9 INA139, x1 jumper, x2 jumper, x3 jumper, x4 jumper, x5 jumper, x6 jumper, x7 jumper, x8 jumper, x9 jumper

Commit message: Pimping PCB
Parts:
- added C75: 330n / 50V, Capacitors_SMD:C_0805, B.Cu at (36.8, 204.5)
- added C76: 47u/16V, Capacitors_SMD:CP_Elec_4x5.8, B.Cu at (41.9, 208.3)
- added C82: 1u/50V, Capacitors_SMD:C_1206, F.Cu at (91.4, 208.8)
- added C83: 1u/50V, Capacitors_SMD:C_1206, F.Cu at (91.9, 140.2)
- added C84: 1u/50V, Capacitors_SMD:C_1206, F.Cu at (103.1, 174.0)
- added C85: 1u/50V, Capacitors_SMD:C_1206, F.Cu at (59.9, 103.6)
- added C86: 1u/50V, Capacitors_SMD:C_1206, F.Cu at (118.4, 103.6)
- added J11: PowerLED, Connectors_JST:JST_XH_B02B-XH-A_02x2.50mm_Straight, F.Cu at (38.7, 209.6)
- added R99: 1k, Resistors_SMD:R_0805, B.Cu at (33.7, 212.1)
- added U17: L78L05_SOT89, TO_SOT_Packages_SMD:SOT-89-3, B.Cu at (33.6, 208.3)
- moved C60 3.81 mm to (142.9, 96.3)
- moved J9 3.81 mm to (137.2, 83.8)
- moved R74 3.81 mm to (135.3, 78.1)
- moved R75 3.81 mm to (133.3, 80.0)
- moved R80 3.81 mm to (141.6, 93.1)
- moved R81 3.81 mm to (145.4, 93.1)
- moved R83 3.81 mm to (146.1, 95.0)
- moved U14 3.81 mm to (143.5, 93.1)
- moved R79 3.81 mm to (137.8, 93.1)
- moved C35 2.55 mm to (113.0, 173.7)
- moved C8 2.55 mm to (106.7, 147.6)
- moved R14 2.55 mm to (109.9, 150.1)
- moved R15 2.55 mm to (108.0, 150.7)
- moved R18 2.55 mm to (109.9, 146.3)
- moved R19 2.55 mm to (109.9, 142.5)
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Connections:
- net Net-(F1-Pad1) renamed Unfused_Power
Routing:
- net GNDA: track 463.8 -> 488.3 mm
- net Net-(C76-Pad1): track 0.00 -> 15.1 mm
- net Unfused_Power: track 0.00 -> 13.1 mm
- net Net-(C10-Pad1): track 40.0 -> 45.6 mm
- net (no net): track 149.1 -> 144.0 mm
- net Net-(C33-Pad1): track 41.2 -> 45.6 mm
- net GND: track 374.6 -> 378.9 mm
- net OUT_1_Current: track 168.1 -> 165.4 mm
- net Net-(R99-Pad2): track 0.00 -> 2.56 mm
- net Net-(C52-Pad1): track 35.7 -> 38.2 mm
- net OUT_2_Current: track 193.3 -> 190.7 mm
- net Net-(C34-Pad1): track 41.1 -> 43.6 mm
- net Net-(C51-Pad1): track 38.8 -> 40.9 mm
- net OUT_3_Current: track 237.0 -> 235.0 mm
- net OUT_5_Current: track 66.8 -> 65.2 mm
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Other:
- board text added: "MobilePowerBank v1 JP, 2018.12.15"
- board text removed: "MobilePowerSupply v1 JP, 2018.10.15"

Commit message: Pimping PCB
Parts:
- moved x4 1.02 mm to (35.6, 96.5)
- moved R98 0.95 mm to (47.6, 42.2)
Routing:
- net (no net): track 144.0 -> 210.0 mm
- net POWER_IN_4: track 90.7 -> 89.7 mm
- net GNDA: track 488.3 -> 489.2 mm
- net GND: track 378.9 -> 377.9 mm
Other:
- board text added: "MobilePowerBank v1 JP, 2018.12.19"
- board text removed: "MobilePowerBank v1 JP, 2018.12.15"

Commit message: DMA and screen
Parts:
- R44: value 90k -> 47k
- R45: value 10k -> 3k9
Changed lines of the file:
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@@
   )
   (setup
-    (last_trace_width 1.6256)
+    (last_trace_width 0.6096)
     (user_trace_width 0.508)
     (user_trace_width 0.6096)
@@
     (add_net SWITCH)
   )
+  (module Inductors_SMD:L_1206 (layer B.Cu)
+    (at 135.89 47.371 270)
+    (descr "Resistor SMD 1206, reflow soldering, Vishay (see dcrcw.pdf)")
+    (tags "resistor 1206")
+    (attr smd)
+    (fp_text reference L1 (at 0 2.3 270) (layer B.SilkS)
+      (effects (font (size 1 1) (thickness 0.15)) (justify mirror))
+    )
+    (fp_text value 10u (at 0 -2.3 270) (layer B.Fab)
+      (effects (font (size 1 1) (thickness 0.15)) (justify mirror))
+    )
+    (fp_text user %R (at 0 0 270) (layer B.Fab)
+      (effects (font (size 0.5 0.5) (thickness 0.075)) (justify mirror))
+    )
+    (fp_line (start -1.6 -0.8) (end -1.6 0.8) (layer B.Fab) (width 0.1))
+    (fp_line (start 1.6 -0.8) (end -1.6 -0.8) (layer B.Fab) (width 0.1))
+    (fp_line (start 1.6 0.8) (end 1.6 -0.8) (layer B.Fab) (width 0.1))
+    (fp_line (start -1.6 0.8) (end 1.6 0.8) (layer B.Fab) (width 0.1))
+    (fp_line (start -2.2 1.2) (end 2.2 1.2) (layer B.CrtYd) (width 0.05))
+    (fp_line (start -2.2 -1.2) (end 2.2 -1.2) (layer B.CrtYd) (width 0.05))
+    (fp_line (start -2.2 1.2) (end -2.2 -1.2) (layer B.CrtYd) (width 0.05))
+    (fp_line (start 2.2 1.2) (end 2.2 -1.2) (layer B.CrtYd) (width 0.05))
+    (fp_line (start 1 -1.07) (end -1 -1.07) (layer B.SilkS) (width 0.12))
+    (fp_line (start -1 1.07) (end 1 1.07) (layer B.SilkS) (width 0.12))
+    (pad 1 smd rect (at -1.45 0 270) (size 0.9 1.7) (layers B.Cu B.Paste B.Mask)
+      (net 15 +3V3))
+    (pad 2 smd rect (at 1.45 0 270) (size 0.9 1.7) (layers B.Cu B.Paste B.Mask)
+      (net 37 /+3.3VA))
+    (model ${KISYS3DMOD}/Inductors_SMD.3dshapes/L_1206.wrl
+      (at (xyz 0 0 0))
+      (scale (xyz 1 1 1))
+      (rotate (xyz 0 0 0))
+    )
+  )
   (module Resistors_SMD:R_0805 (layer B.Cu)
     (at 91.76 38.227 180)
@@
       (effects (font (size 1 1) (thickness 0.15)) (justify mirror))
     )
-    (fp_text value 90k (at 0 -1.75 90) (layer B.Fab)
+    (fp_text value 47k (at 0 -1.75 90) (layer B.Fab)
       (effects (font (size 1 1) (thickness 0.15)) (justify mirror))
     )
@@
       (effects (font (size 1 1) (thickness 0.15)) (justify mirror))
     )
-    (fp_text value 10k (at 0 -1.75 90) (layer B.Fab)
+    (fp_text value 3k9 (at 0 -1.75 90) (layer B.Fab)
       (effects (font (size 1 1) (thickness 0.15)) (justify mirror))
     )
@@
       (at (xyz 0 0 0))
       (scale (xyz 1 1 1))
-      (rotate (xyz 0 0 0))
-    )
-  )
-  (module Inductors_SMD:L_1206 (layer B.Cu)
-    (at 135.89 47.371 270)
-    (descr "Resistor SMD 1206, reflow soldering, Vishay (see dcrcw.pdf)")
-    (tags "resistor 1206")
-    (attr smd)
-    (fp_text reference L1 (at 0 2.3 270) (layer B.SilkS)
-      (effects (font (size 1 1) (thickness 0.15)) (justify mirror))
-    )
-    (fp_text value 10u (at 0 -2.3 270) (layer B.Fab)
-      (effects (font (size 1 1) (thickness 0.15)) (justify mirror))
-    )
-    (fp_text user %R (at 0 0 270) (layer B.Fab)
-      (effects (font (size 0.5 0.5) (thickness 0.075)) (justify mirror))
-    )
-    (fp_line (start -1.6 -0.8) (end -1.6 0.8) (layer B.Fab) (width 0.1))
-    (fp_line (start 1.6 -0.8) (end -1.6 -0.8) (layer B.Fab) (width 0.1))
-    (fp_line (start 1.6 0.8) (end 1.6 -0.8) (layer B.Fab) (width 0.1))
-    (fp_line (start -1.6 0.8) (end 1.6 0.8) (layer B.Fab) (width 0.1))
-    (fp_line (start -2.2 1.2) (end 2.2 1.2) (layer B.CrtYd) (width 0.05))
-    (fp_line (start -2.2 -1.2) (end 2.2 -1.2) (layer B.CrtYd) (width 0.05))
-    (fp_line (start -2.2 1.2) (end -2.2 -1.2) (layer B.CrtYd) (width 0.05))
-    (fp_line (start 2.2 1.2) (end 2.2 -1.2) (layer B.CrtYd) (width 0.05))
-    (fp_line (start 1 -1.07) (end -1 -1.07) (layer B.SilkS) (width 0.12))
-    (fp_line (start -1 1.07) (end 1 1.07) (layer B.SilkS) (width 0.12))
-    (pad 1 smd rect (at -1.45 0 270) (size 0.9 1.7) (layers B.Cu B.Paste B.Mask)
-      (net 15 +3V3))
-    (pad 2 smd rect (at 1.45 0 270) (size 0.9 1.7) (layers B.Cu B.Paste B.Mask)
-      (net 37 /+3.3VA))
-    (model ${KISYS3DMOD}/Inductors_SMD.3dshapes/L_1206.wrl
-      (at (xyz 0 0 0))
-      (scale (xyz 1 1 1))

Commit message: Five outputs callibration
Parts:
- C76: value 47u/16V -> 22u/16V
- R12: value 90k -> 100k
- R13: value 10k -> 4k7
- R99: value 1k -> 3k3
Connections:
- J5 pad 3: (no net) -> Net-(J5-Pad3)
- J5 pad 4: (no net) -> Net-(J5-Pad4)
- J6 pad 18: (no net) -> Net-(J6-Pad18)
- J6 pad 22: (no net) -> Net-(J6-Pad22)
- J6 pad 23: (no net) -> Net-(J6-Pad23)
- J6 pad 24: (no net) -> Net-(J6-Pad24)
- J6 pad 25: (no net) -> Net-(J6-Pad25)
- J6 pad 26: (no net) -> Net-(J6-Pad26)
- J6 pad 27: (no net) -> Net-(J6-Pad27)
- J6 pad 28: (no net) -> Net-(J6-Pad28)
- J6 pad 30: (no net) -> Net-(J6-Pad30)
- U15 pad 13: (no net) -> Net-(U15-Pad13)
- U15 pad 18: (no net) -> Net-(U15-Pad18)
- U15 pad 19: (no net) -> Net-(U15-Pad19)
- U15 pad 20: (no net) -> Net-(U15-Pad20)
- U15 pad 21: (no net) -> Net-(U15-Pad21)
- U15 pad 22: (no net) -> Net-(U15-Pad22)
- U15 pad 23: (no net) -> Net-(U15-Pad23)
- U15 pad 26: (no net) -> Net-(U15-Pad26)
- U15 pad 27: (no net) -> Net-(U15-Pad27)
- U15 pad 33: (no net) -> Net-(U15-Pad33)
- U15 pad 46: (no net) -> Net-(U15-Pad46)
- U15 pad 47: (no net) -> Net-(U15-Pad47)
- U15 pad 50: (no net) -> Net-(U15-Pad50)
- U15 pad 51: (no net) -> Net-(U15-Pad51)
- U15 pad 54: (no net) -> Net-(U15-Pad54)
- U15 pad 55: (no net) -> Net-(U15-Pad55)
- U15 pad 58: (no net) -> Net-(U15-Pad58)
- U15 pad 59: (no net) -> Net-(U15-Pad59)
- U15 pad 62: (no net) -> Net-(U15-Pad62)
